Commit message: add a home named robot pose to the arm in moveit setup

File: homestri_robot_description/urdf/base_scene.urdf.xacro (robot description, xacro)
@@ -49,3 +49,30 @@
     <origin xyz="0 0 0" rpy="0 0 0" />
   </joint>
+  <link name="panel">
+  <inertial>
+  <origin xyz="0 0 0" rpy="0 0 0"/>
+  <mass value="1"/>
+    <inertia ixx="100"  ixy="0"  ixz="0" iyy="100" iyz="0" izz="100" />
+    </inertial>
+    <visual>
+      <origin xyz="0 0 0" rpy="0 0 0" />
+      <geometry>
+        <box size="2 2 0.02" />
+      </geometry>
+        <material name="Cyan">
+      <color rgba="0 1.0 1.0 1.0"/>
+        </material>
+    </visual>
+    <collision>
+      <origin xyz="0 0 0" rpy="0 0 0"/>
+        <geometry>
+          <box size="2 2 0.02" />
+        </geometry>
+    </collision>
+  </link>
+  <joint name="panel_to_world" type="fixed">
+    <parent link="world"/>
+    <child link="panel"/>
+    <origin xyz="0 0 -0.1" />
+  </joint>
 </robot>
