Commit message: update pedestal to match workspace

File: homestri_robot_description/urdf/base_scene.xacro (robot description, xacro)
@@ -1,10 +1,10 @@
 <?xml version="1.0"?>
 <robot xmlns:xacro="http://www.ros.org/wiki/xacro" name="base_scene">
-  <xacro:include filename="$(find homestri_robot_description)/urdf/environment.xacro" />
+  <xacro:include filename="$(find homestri_robot_description)/urdf/workspace.xacro" />
   <xacro:include filename="$(find homestri_robot_description)/urdf/ur5e_macro.xacro" />
   <xacro:include filename="$(find homestri_robot_description)/urdf/robotiq_2f_85_macro.xacro" />
-  <xacro:environment
-    pedestal_height="0.2"
-    pedestal_radius="0.12"
+  <xacro:workspace
+    pedestal_height="0.145"
+    pedestal_radius="0.1"
   />
   <xacro:ur5e

File: homestri_robot_description/urdf/workspace.xacro (robot description, xacro)
@@ -2,6 +2,6 @@
 <!-- This macro adds a convenient TF frame at the tip of the closed gripper. -->
 <!-- The position of the TF frame has not been measured at all and needs to be calibrated. -->
-<robot name="environment_homestri" xmlns:xacro="http://www.ros.org/wiki/xacro">
-  <xacro:macro name="environment" params="pedestal_height:=0.2 pedestal_radius:=0.2">
+<robot name="workspace_homestri" xmlns:xacro="http://www.ros.org/wiki/xacro">
+  <xacro:macro name="workspace" params="pedestal_height:=0.2 pedestal_radius:=0.2">
     <link name="pedestal">
       <visual>

Commit message: new urdf table (bare bones), homestri_bringup package for easy bringup/calibration

File: homestri_robot_description/urdf/base_scene.xacro (robot description, xacro)
@@ -10,8 +10,8 @@
   <xacro:ur5e
     prefix=""
-    parent="pedestal"
+    parent="ground"
     transmission_hw_interface="hardware_interface/PositionJointInterface"
   >
-    <origin xyz="0 0 0" rpy="0 0 0" />
+    <origin xyz="0 0 -0.025" rpy="0 0 0" />
   </xacro:ur5e>
   <xacro:robotiq_2f_85

File: homestri_robot_description/urdf/workspace.xacro (robot description, xacro)
@@ -4,5 +4,5 @@
 <robot name="workspace_homestri" xmlns:xacro="http://www.ros.org/wiki/xacro">
   <xacro:macro name="workspace" params="pedestal_height:=0.2 pedestal_radius:=0.2">
-    <link name="pedestal">
+    <!-- <link name="pedestal">
       <visual>
         <origin rpy="0 0 0" xyz="0 0 ${-pedestal_height/2}"/>
@@ -20,5 +20,4 @@
         </geometry>
       </collision>
-      <!-- these are dummy intertial values to spawn the object in gazebo -->
       <inertial>
         <origin xyz="0.0 0.0 0.02" rpy="0 0 0" />
@@ -26,5 +25,5 @@
         <inertia ixx=".18e-05" iyy=".18e-05" izz=".18e-05" ixy="0.0" iyz="0.0" ixz="0.0" />
       </inertial>
-    </link>
+    </link> -->
     <link name="ground">
         <collision>
@@ -35,9 +34,9 @@
         </collision>
     </link>
-    <joint name="pedestal_to_world" type="fixed">
+    <!-- <joint name="pedestal_to_world" type="fixed">
         <parent link="world"/>
         <child link="pedestal"/>
         <origin xyz="0 0 ${pedestal_height}" />
-    </joint>
+    </joint> -->
     <joint name="ground_to_world" type="fixed">
         <parent link="world"/>

Commit message: updated table workspace (table flush with robot base)

File: homestri_robot_description/urdf/base_scene.xacro (robot description, xacro)
@@ -4,14 +4,11 @@
   <xacro:include filename="$(find homestri_robot_description)/urdf/ur5e_macro.xacro" />
   <xacro:include filename="$(find homestri_robot_description)/urdf/robotiq_2f_85_macro.xacro" />
-  <xacro:workspace
-    pedestal_height="0.135"
-    pedestal_radius="0.1"
-  />
+  <xacro:workspace />
   <xacro:ur5e
     prefix=""
-    parent="ground"
+    parent="world"
     transmission_hw_interface="hardware_interface/PositionJointInterface"
   >
-    <origin xyz="0 0 -0.025" rpy="0 0 0" />
+    <origin xyz="0 0 0" rpy="0 0 0" />
   </xacro:ur5e>
   <xacro:robotiq_2f_85

File: homestri_robot_description/urdf/workspace.xacro (robot description, xacro)
@@ -3,5 +3,6 @@
 <!-- The position of the TF frame has not been measured at all and needs to be calibrated. -->
 <robot name="workspace_homestri" xmlns:xacro="http://www.ros.org/wiki/xacro">
-  <xacro:macro name="workspace" params="pedestal_height:=0.2 pedestal_radius:=0.2">
+  <xacro:macro name="workspace">
+  <!-- <xacro:macro name="workspace" params="pedestal_height:=0.2 pedestal_radius:=0.2"> -->
     <!-- <link name="pedestal">
       <visual>
