Commit message: added scene manager

File: homestri_robot_description/urdf/parts/box.xacro (robot description, xacro)
@@ -1,4 +1,5 @@
 <?xml version="1.0"?>
-<robot name="red_box">
+<robot xmlns:xacro="http://www.ros.org/wiki/xacro" name="box">
+  <xacro:arg name="color" default="255 255 255 1"/>
   <link name="base_link">
     <collision>
@@ -26,6 +27,6 @@
     <visual>
       <material>
-        <ambient>0.3137254 0.3254902 0.2352941 1</ambient>
-        <diffuse>0.3137254 0.3254902 0.2352941 1</diffuse>
+        <ambient>$(arg color)</ambient>
+        <diffuse>$(arg color)</diffuse>
         <specular>0.1 0.1 0.1 1</specular>
         <emissive>0 0 0 0</emissive>

File: homestri_robot_description/urdf/parts/plastic_bin.xacro (robot description, xacro)
@@ -1,4 +1,4 @@
 <?xml version="1.0"?>
-<robot name="plastic_bin">
+<robot xmlns:xacro="http://www.ros.org/wiki/xacro" name="plastic_bin">
   <link name="base_link">
     <inertial>
@@ -24,5 +24,12 @@
   </link>
   <gazebo reference="base_link">
-    <material>Gazebo/Green</material>
+    <visual>
+      <material>
+        <ambient>$(arg color)</ambient>
+        <diffuse>$(arg color)</diffuse>
+        <specular>0.1 0.1 0.1 1</specular>
+        <emissive>0 0 0 0</emissive>
+      </material>
+    </visual>
     <kp>1000000.0</kp>
     <kd>1.0</kd>
