Commit message: reran moveit setup assistant

File: homestri_moveit_config/config/gazebo_base_scene.urdf (robot description, URDF)
Before this commit: robot base_scene, 25 links, 24 joints
Links:
- removed link a_bot_base
- removed link a_bot_base_link
- removed link a_bot_base_link_inertia
- removed link a_bot_ee_link
- removed link a_bot_flange
- removed link a_bot_forearm_link
- removed link a_bot_gripper_tip_link
- removed link a_bot_left_inner_finger
- removed link a_bot_left_inner_finger_pad
- removed link a_bot_left_inner_knuckle
- removed link a_bot_left_outer_finger
- removed link a_bot_left_outer_knuckle
- removed link a_bot_right_inner_finger
- removed link a_bot_right_inner_finger_pad
- removed link a_bot_right_inner_knuckle
- removed link a_bot_right_outer_finger
- removed link a_bot_right_outer_knuckle
- removed link a_bot_robotiq_arg2f_base_link
- removed link a_bot_shoulder_link
- removed link a_bot_tool0
- removed link a_bot_upper_arm_link
- removed link a_bot_wrist_1_link
- removed link a_bot_wrist_2_link
- removed link a_bot_wrist_3_link
- added link base
- added link base_link
- added link base_link_inertia, mass 4.0; collision mesh filename=package://ur_description/meshes/ur5e/collision/base.stl; visual mesh filename=package://ur_description/meshes/ur5e/visual/base.dae
- added link ee_link, mass 0.1; collision box size=0.01 0.01 0.01
- added link flange
- added link forearm_link, mass 2.275; collision mesh filename=package://ur_description/meshes/ur5e/collision/forearm.stl; visual mesh filename=package://ur_description/meshes/ur5e/visual/forearm.dae
- added link gripper_tip_link
- added link left_inner_finger, mass 0.0104003125914103; collision mesh filename=package://robotiq_2f_85_gripper_visualization/meshes/collis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 scale=0.001 0.001 0.001; visual mesh filename=package://robotiq_2f_85_gripper_visualization/meshes/visual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 scale=0.001 0.001 0.001
- added link left_inner_finger_pad, mass 0.1; collision box size=0.022 0.00635 0.0375; visual box size=0.022 0.00635 0.0375
- added link left_inner_knuckle, mass 0.0271177346495152; collision mesh filename=package://robotiq_2f_85_gripper_visualization/meshes/collis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 scale=0.001 0.001 0.001; visual mesh filename=package://robotiq_2f_85_gripper_visualization/meshes/visual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 scale=0.001 0.001 0.001
- added link left_outer_finger, mass 0.022614240507152; collision mesh filename=package://robotiq_2f_85_gripper_visualization/meshes/collis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 scale=0.001 0.001 0.001; visual mesh filename=package://robotiq_2f_85_gripper_visualization/meshes/visual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 scale=0.001 0.001 0.001
- added link left_outer_knuckle, mass 0.00853198276973456; collision mesh filename=package://robotiq_2f_85_gripper_visualization/meshes/collis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 scale=0.001 0.001 0.001; visual mesh filename=package://robotiq_2f_85_gripper_visualization/meshes/visual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 scale=0.001 0.001 0.001
- added link right_inner_finger, mass 0.0104003125914103; collision mesh filename=package://robotiq_2f_85_gripper_visualization/meshes/collis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 scale=0.001 0.001 0.001; visual mesh filename=package://robotiq_2f_85_gripper_visualization/meshes/visual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 scale=0.001 0.001 0.001
- added link right_inner_finger_pad, mass 0.1; collision box size=0.022 0.00635 0.0375; visual box size=0.022 0.00635 0.0375
- added link right_inner_knuckle, mass 0.0271177346495152; collision mesh filename=package://robotiq_2f_85_gripper_visualization/meshes/collis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 scale=0.001 0.001 0.001; visual mesh filename=package://robotiq_2f_85_gripper_visualization/meshes/visual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 scale=0.001 0.001 0.001
- added link right_outer_finger, mass 0.022614240507152; collision mesh filename=package://robotiq_2f_85_gripper_visualization/meshes/collis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 scale=0.001 0.001 0.001; visual mesh filename=package://robotiq_2f_85_gripper_visualization/meshes/visual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 scale=0.001 0.001 0.001
- added link right_outer_knuckle, mass 0.00853198276973456; collision mesh filename=package://robotiq_2f_85_gripper_visualization/meshes/collis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 scale=0.001 0.001 0.001; visual mesh filename=package://robotiq_2f_85_gripper_visualization/meshes/visual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 scale=0.001 0.001 0.001
- added link robotiq_arg2f_base_link, mass 0.22652; collision mesh filename=package://robotiq_2f_85_gripper_visualization/meshes/collis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; visual mesh filename=package://robotiq_2f_85_gripper_visualization/meshes/visual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
- added link shoulder_link, mass 3.7; collision mesh filename=package://ur_description/meshes/ur5e/collision/shoulder.stl; visual mesh filename=package://ur_description/meshes/ur5e/visual/shoulder.dae
- added link tool0
- added link upper_arm_link, mass 8.393; collision mesh filename=package://ur_description/meshes/ur5e/collision/upperarm.stl; visual mesh filename=package://ur_description/meshes/ur5e/visual/upperarm.dae
- added link wrist_1_link, mass 1.219; collision mesh filename=package://ur_description/meshes/ur5e/collision/wrist1.stl; visual mesh filename=package://ur_description/meshes/ur5e/visual/wrist1.dae
- added link wrist_2_link, mass 1.219; collision mesh filename=package://ur_description/meshes/ur5e/collision/wrist2.stl; visual mesh filename=package://ur_description/meshes/ur5e/visual/wrist2.dae
- added link wrist_3_link, mass 0.1879; collision mesh filename=package://ur_description/meshes/ur5e/collision/wrist3.stl; visual mesh filename=package://ur_description/meshes/ur5e/visual/wrist3.dae
Joints:
- removed joint a_bot_base_link-base_fixed_joint
- removed joint a_bot_base_link-base_link_inertia
- removed joint a_bot_ee_fixed_joint
- removed joint a_bot_elbow_joint
- removed joint a_bot_finger_joint
- removed joint a_bot_flange-tool0
- removed joint a_bot_gripper_tip_link_joint
- removed joint a_bot_left_inner_finger_joint
- removed joint a_bot_left_inner_finger_pad_joint
- removed joint a_bot_left_inner_knuckle_joint
- removed joint a_bot_left_outer_finger_joint
- removed joint a_bot_right_finger_joint
- removed joint a_bot_right_inner_finger_joint
- removed joint a_bot_right_inner_finger_pad_joint
- removed joint a_bot_right_inner_knuckle_joint
- removed joint a_bot_right_outer_finger_joint
- removed joint a_bot_robotiq_85_base_joint
- removed joint a_bot_shoulder_lift_joint
- removed joint a_bot_shoulder_pan_joint
- removed joint a_bot_wrist_1_joint
- removed joint a_bot_wrist_2_joint
- removed joint a_bot_wrist_3-flange
- removed joint a_bot_wrist_3_joint
- removed joint world_a_bot_joint
- added joint base_link-base_fixed_joint: type fixed, parent base_link, child base, origin xyz=0 0 0 rpy=0 0 3.141592653589793
- added joint base_link-base_link_inertia: type fixed, parent base_link, child base_link_inertia, origin xyz=0 0 0 rpy=0 0 3.141592653589793
- added joint ee_fixed_joint: type fixed, parent wrist_3_link, child ee_link, origin xyz=0.0 0.0 0.0 rpy=0.0 -1.57079632679 1.57079632679
- added joint elbow_joint: type revolute, parent upper_arm_link, child forearm_link, origin xyz=-0.425 0 0 rpy=0 0 0, axis 0 0 1, limit lower=-3.141592653589793 upper=3.141592653589793 effort=150.0 velocity=3.141592653589793
- added joint finger_joint: type revolute, parent robotiq_arg2f_base_link, child left_outer_knuckle, origin xyz=0 -0.0306011 0.054904 rpy=0 0 3.141592653589793, axis 1 0 0, limit lower=0 upper=0.8 effort=1000 velocity=0.5
- added joint flange-tool0: type fixed, parent flange, child tool0, origin xyz=0 0 0 rpy=1.5707963267948966 0 1.5707963267948966
- added joint gripper_tip_link_joint: type fixed, parent ee_link, child gripper_tip_link, origin xyz=0.163 0 0 rpy=0 0 0
- added joint left_inner_finger_joint: type revolute, parent left_outer_finger, child left_inner_finger, origin xyz=0 0.0061 0.0471 rpy=0 0 0, axis 1 0 0, limit lower=-0.8757 upper=0 effort=1000 velocity=0.5, mimic joint=finger_joint multiplier=-1 offset=0
- added joint left_inner_finger_pad_joint: type fixed, parent left_inner_finger, child left_inner_finger_pad, origin xyz=0 -0.0220203446692936 0.03242 rpy=0 0 0, axis 0 0 1
- added joint left_inner_knuckle_joint: type revolute, parent robotiq_arg2f_base_link, child left_inner_knuckle, origin xyz=0 -0.0127 0.06142 rpy=0 0 3.141592653589793, axis 1 0 0, limit lower=0 upper=0.8757 effort=1000 velocity=0.5, mimic joint=finger_joint multiplier=1 offset=0
- added joint left_outer_finger_joint: type fixed, parent left_outer_knuckle, child left_outer_finger, origin xyz=0 0.0315 -0.0041 rpy=0 0 0, axis 1 0 0
- added joint right_finger_joint: type revolute, parent robotiq_arg2f_base_link, child right_outer_knuckle, origin xyz=0 0.0306011 0.054904 rpy=0 0 0, axis 1 0 0, limit lower=0 upper=0.81 effort=1000 velocity=0.5, mimic joint=finger_joint multiplier=1 offset=0
- added joint right_inner_finger_joint: type revolute, parent right_outer_finger, child right_inner_finger, origin xyz=0 0.0061 0.0471 rpy=0 0 0, axis 1 0 0, limit lower=-0.8757 upper=0 effort=1000 velocity=0.5, mimic joint=finger_joint multiplier=-1 offset=0
- added joint right_inner_finger_pad_joint: type fixed, parent right_inner_finger, child right_inner_finger_pad, origin xyz=0 -0.0220203446692936 0.03242 rpy=0 0 0, axis 0 0 1
- added joint right_inner_knuckle_joint: type revolute, parent robotiq_arg2f_base_link, child right_inner_knuckle, origin xyz=0 0.0127 0.06142 rpy=0 0 0.0, axis 1 0 0, limit lower=0 upper=0.8757 effort=1000 velocity=0.5, mimic joint=finger_joint multiplier=1 offset=0
- added joint right_outer_finger_joint: type fixed, parent right_outer_knuckle, child right_outer_finger, origin xyz=0 0.0315 -0.0041 rpy=0 0 0, axis 1 0 0
- added joint robotiq_85_base_joint: type fixed, parent ee_link, child robotiq_arg2f_base_link, origin xyz=0 0 0 rpy=3.141592653589793 -1.5707963267948966 0
- added joint shoulder_lift_joint: type revolute, parent shoulder_link, child upper_arm_link, origin xyz=0 0 0 rpy=1.570796327 0 0, axis 0 0 1, limit lower=-6.283185307179586 upper=6.283185307179586 effort=150.0 velocity=3.141592653589793
- added joint shoulder_pan_joint: type revolute, parent base_link_inertia, child shoulder_link, origin xyz=0 0 0.1625 rpy=0 0 0, axis 0 0 1, limit lower=-6.283185307179586 upper=6.283185307179586 effort=150.0 velocity=3.141592653589793
- added joint world_joint: type fixed, parent world, child base_link, origin xyz=0 0 0 rpy=0 0 0
- added joint wrist_1_joint: type revolute, parent forearm_link, child wrist_1_link, origin xyz=-0.3922 0 0.1333 rpy=0 0 0, axis 0 0 1, limit lower=-6.283185307179586 upper=6.283185307179586 effort=28.0 velocity=3.141592653589793
- added joint wrist_2_joint: type revolute, parent wrist_1_link, child wrist_2_link, origin xyz=0 -0.0997 -2.044881182297852e-11 rpy=1.570796327 0 0, axis 0 0 1, limit lower=-6.283185307179586 upper=6.283185307179586 effort=28.0 velocity=3.141592653589793
- added joint wrist_3-flange: type fixed, parent wrist_3_link, child flange, origin xyz=0 0 0 rpy=0 -1.5707963267948966 -1.5707963267948966
- added joint wrist_3_joint: type revolute, parent wrist_2_link, child wrist_3_link, origin xyz=0 0.0996 -2.042830148012698e-11 rpy=1.570796326589793 3.141592653589793 3.141592653589793, axis 0 0 1, limit lower=-6.283185307179586 upper=6.283185307179586 effort=28.0 velocity=3.141592653589793

File: homestri_robot_description/urdf/base_scene.urdf.xacro (robot description, xacro)
@@ -4,5 +4,5 @@
   <xacro:include filename="$(find ur_description)/urdf/inc/ur_macro.xacro"/>
   <xacro:ur_robot
-    prefix="a_bot_"
+    prefix=""
     joint_limits_parameters_file='$(find ur_description)/config/ur5e/joint_limits.yaml'
     kinematics_parameters_file='$(find ur_description)/config/ur5e/default_kinematics.yaml'
@@ -14,5 +14,5 @@
     safety_k_position="20"
   />
-  <link name="a_bot_ee_link">
+  <link name="ee_link">
     <collision>
       <geometry>
@@ -22,29 +22,29 @@
     </collision>
   </link>
-  <joint name="a_bot_ee_fixed_joint" type="fixed">
-    <parent link="a_bot_wrist_3_link"/>
-    <child link="a_bot_ee_link"/>
+  <joint name="ee_fixed_joint" type="fixed">
+    <parent link="wrist_3_link"/>
+    <child link="ee_link"/>
     <origin rpy="0.0 -1.57079632679 1.57079632679" xyz="0.0 0.0 0.0"/>
   </joint>
   <!-- Spawn and attach robotiq 85 gripper (+ cameras) -->
   <xacro:include filename="$(find robotiq_2f_85_gripper_visualization)/urdf/robotiq_arg2f_85_macro.xacro" />
-  <xacro:robotiq_arg2f_85 prefix="a_bot_" transmission_hw_interface="hardware_interface/EffortJointInterface"/>
-  <joint name="a_bot_robotiq_85_base_joint" type="fixed">
-    <parent link="a_bot_ee_link"/>
-    <child link="a_bot_robotiq_arg2f_base_link"/>
+  <xacro:robotiq_arg2f_85 prefix="" transmission_hw_interface="hardware_interface/EffortJointInterface"/>
+  <joint name="robotiq_85_base_joint" type="fixed">
+    <parent link="ee_link"/>
+    <child link="robotiq_arg2f_base_link"/>
     <origin xyz="0 0 0" rpy="${pi} ${-pi/2} 0" />
     <!-- <origin xyz="0.01 0 0" rpy="${pi} ${-pi/2} 0" /> -->
   </joint>
   <!-- Add an additional link to plan with. Oriented like the UR ee_link frame. -->
-  <link name="a_bot_gripper_tip_link"/>
-  <joint name="a_bot_gripper_tip_link_joint" type="fixed">
-    <parent link="a_bot_ee_link"/>
-    <child link="a_bot_gripper_tip_link"/>
+  <link name="gripper_tip_link"/>
+  <joint name="gripper_tip_link_joint" type="fixed">
+    <parent link="ee_link"/>
+    <child link="gripper_tip_link"/>
     <origin rpy="0 0 0" xyz="0.163 0 0"/>
   </joint>
   <link name="world" />
-  <joint name="world_a_bot_joint" type="fixed">
+  <joint name="world_joint" type="fixed">
     <parent link="world" />
-    <child link="a_bot_base_link" />
+    <child link="base_link" />
     <origin xyz="0 0 0" rpy="0 0 0" />
   </joint>

Commit message: added pedestal, table, coupling. Changed joint limits. Updated moveit_config

File: homestri_moveit_config/config/gazebo_base_scene.urdf (robot description, URDF)
Before this commit: robot base_scene, 25 links, 24 joints
Links:
- added link coupling, mass 0.1; collision cylinder length=0.01 radius=0.0375; visual cylinder length=0.01 radius=0.0375
- added link pedestal, mass 0.1; collision cylinder length=0.2 radius=0.2; visual cylinder length=0.2 radius=0.2
- added link table, mass 0.1; collision box size=3 3 0.02; visual box size=3 3 0.02
Joints:
- added joint arm_to_pedestal: type fixed, parent pedestal, child base_link, origin xyz=0 0 0 rpy=0 0 0
- added joint coupling_joint: type fixed, parent ee_link, child coupling, origin xyz=0 0 0 rpy=0 0 0
- added joint pedestal_to_table: type fixed, parent table, child pedestal, origin xyz=0 0 0.22
- joint elbow_joint: limit lower=-3.141592653589793 upper=3.141592653589793 effort=150.0 velocity=3.141592653589793 -> lower=0.0 upper=3.141592653589793 effort=150.0 velocity=3.141592653589793
- joint robotiq_85_base_joint: origin xyz=0 0 0 rpy=3.141592653589793 -1.5707963267948966 0 -> xyz=0.01 0 0 rpy=3.141592653589793 -1.5707963267948966 0
- joint shoulder_lift_joint: limit lower=-6.283185307179586 upper=6.283185307179586 effort=150.0 velocity=3.141592653589793 -> lower=-3.141592653589793 upper=3.141592653589793 effort=150.0 velocity=3.141592653589793
- joint shoulder_pan_joint: limit lower=-6.283185307179586 upper=6.283185307179586 effort=150.0 velocity=3.141592653589793 -> lower=-3.141592653589793 upper=3.141592653589793 effort=150.0 velocity=3.141592653589793
- joint world_joint: child base_link -> table
- joint wrist_1_joint: limit lower=-6.283185307179586 upper=6.283185307179586 effort=28.0 velocity=3.141592653589793 -> lower=-4.71238898038469 upper=3.141592653589793 effort=28.0 velocity=3.141592653589793
- joint wrist_2_joint: limit lower=-6.283185307179586 upper=6.283185307179586 effort=28.0 velocity=3.141592653589793 -> lower=-4.71238898038469 upper=4.71238898038469 effort=28.0 velocity=3.141592653589793

File: homestri_robot_description/urdf/base_scene.urdf.xacro (robot description, xacro)
@@ -2,49 +2,21 @@
 <robot xmlns:xacro="http://www.ros.org/wiki/xacro"
        name="base_scene" >
-  <xacro:include filename="$(find ur_description)/urdf/inc/ur_macro.xacro"/>
-  <xacro:ur_robot
-    prefix=""
-    joint_limits_parameters_file='$(find ur_description)/config/ur5e/joint_limits.yaml'
-    kinematics_parameters_file='$(find ur_description)/config/ur5e/default_kinematics.yaml'
-    physical_parameters_file='$(find ur_description)/config/ur5e/physical_parameters.yaml'
-    visual_parameters_file='$(find ur_description)/config/ur5e/visual_parameters.yaml'
-    transmission_hw_interface='hardware_interface/PositionJointInterface'
-    safety_limits="false"
-    safety_pos_margin="0.15"
-    safety_k_position="20"
-  />
-  <link name="ee_link">
-    <collision>
-      <geometry>
-        <box size="0.01 0.01 0.01"/>
-      </geometry>
-      <origin rpy="0 0 0" xyz="-0.01 0 0"/>
-    </collision>
-  </link>
-  <joint name="ee_fixed_joint" type="fixed">
-    <parent link="wrist_3_link"/>
-    <child link="ee_link"/>
-    <origin rpy="0.0 -1.57079632679 1.57079632679" xyz="0.0 0.0 0.0"/>
+  <!-- ur5e arm and robotiq gripper -->
+  <xacro:include filename="$(find homestri_robot_description)/urdf/ur5e_robotiq.urdf.xacro" />
+  <xacro:ur5e_robotiq />
+  <!-- scene environment (pedestal and table) -->
+  <xacro:include filename="$(find homestri_robot_description)/urdf/environment.urdf.xacro" />
+  <xacro:environment />
+  <!-- attach arm to pedestal. -->
+  <joint name="arm_to_pedestal" type="fixed">
+    <parent link="pedestal" />
+    <child link="base_link" />
+    <origin xyz="0 0 0" rpy="0 0 0" />
   </joint>
-  <!-- Spawn and attach robotiq 85 gripper (+ cameras) -->
-  <xacro:include filename="$(find robotiq_2f_85_gripper_visualization)/urdf/robotiq_arg2f_85_macro.xacro" />
-  <xacro:robotiq_arg2f_85 prefix="" transmission_hw_interface="hardware_interface/EffortJointInterface"/>
-  <joint name="robotiq_85_base_joint" type="fixed">
-    <parent link="ee_link"/>
-    <child link="robotiq_arg2f_base_link"/>
-    <origin xyz="0 0 0" rpy="${pi} ${-pi/2} 0" />
-    <!-- <origin xyz="0.01 0 0" rpy="${pi} ${-pi/2} 0" /> -->
-  </joint>
-  <!-- Add an additional link to plan with. Oriented like the UR ee_link frame. -->
-  <link name="gripper_tip_link"/>
-  <joint name="gripper_tip_link_joint" type="fixed">
-    <parent link="ee_link"/>
-    <child link="gripper_tip_link"/>
-    <origin rpy="0 0 0" xyz="0.163 0 0"/>
-  </joint>
+  <!-- attach arm to world. -->
   <link name="world" />
   <joint name="world_joint" type="fixed">
     <parent link="world" />
-    <child link="base_link" />
+    <child link="table" />
     <origin xyz="0 0 0" rpy="0 0 0" />
   </joint>
