Commit message: working gazebo, remove pedestal

File: homestri_moveit_config/config/gazebo_base_scene.urdf (robot description, URDF)
Before this commit: robot base_scene, 28 links, 27 joints
Links:
- removed link pedestal
- removed link table
- link left_inner_finger: mass 0.0104003125914103 -> 0.01957844415989899
- link left_inner_finger_pad: mass 0.1 -> 0.014144625000000003
- link left_inner_knuckle: mass 0.0271177346495152 -> 0.029949543712543904
- link left_outer_finger: mass 0.022614240507152 -> 0.02729659380694228
- link left_outer_knuckle: mass 0.00853198276973456 -> 0.018476648450763997
- link right_inner_finger: mass 0.0104003125914103 -> 0.01957844415989899
- link right_inner_finger_pad: mass 0.1 -> 0.014144625000000003
- link right_inner_knuckle: mass 0.0271177346495152 -> 0.029949543712543904
- link right_outer_finger: mass 0.022614240507152 -> 0.02729659380694228
- link right_outer_knuckle: mass 0.00853198276973456 -> 0.018476648450763997
- link robotiq_arg2f_base_link: mass 0.22652 -> 0.22651999999800307
Joints:
- removed joint arm_to_pedestal
- removed joint pedestal_to_table
- joint world_joint: child table -> base_link
- joint wrist_1_joint: limit lower=-4.71238898038469 upper=3.141592653589793 effort=28.0 velocity=3.141592653589793 -> lower=-3.141592653589793 upper=3.141592653589793 effort=28.0 velocity=3.141592653589793
- joint wrist_2_joint: limit lower=-4.71238898038469 upper=4.71238898038469 effort=28.0 velocity=3.141592653589793 -> lower=-3.141592653589793 upper=3.141592653589793 effort=28.0 velocity=3.141592653589793
- joint wrist_3_joint: limit lower=-6.283185307179586 upper=6.283185307179586 effort=28.0 velocity=3.141592653589793 -> lower=-3.141592653589793 upper=3.141592653589793 effort=28.0 velocity=3.141592653589793

File: homestri_robot_description/urdf/base_scene.urdf.xacro (robot description, xacro)
@@ -8,17 +8,11 @@
   <xacro:robotiq_2f_85 prefix="" parent="ee_link" />
   <!-- scene environment (pedestal and table) -->
-  <xacro:include filename="$(find homestri_robot_description)/urdf/environment.urdf.xacro" />
-  <xacro:environment />
-  <!-- attach arm to pedestal. -->
-  <joint name="arm_to_pedestal" type="fixed">
-    <parent link="pedestal" />
-    <child link="base_link" />
-    <origin xyz="0 0 0" rpy="0 0 0" />
-  </joint>
+  <!-- <xacro:include filename="$(find homestri_robot_description)/urdf/environment.urdf.xacro" />
+  <xacro:environment /> -->
   <!-- attach table to world. -->
   <link name="world" />
   <joint name="world_joint" type="fixed">
     <parent link="world" />
-    <child link="table" />
+    <child link="base_link" />
     <origin xyz="0 0 0" rpy="0 0 0" />
   </joint>

File: homestri_robot_description/urdf/parts/box.urdf (robot description, URDF)
Before this commit: robot red_box, 1 links, 0 joints
Links:
- link base_link: mass 0.001 -> .006784

File: homestri_robot_description/urdf/robotiq_2f_85_macro.urdf.xacro (robot description, xacro)
@@ -2,13 +2,15 @@
 <!-- This macro adds a convenient TF frame at the tip of the closed gripper. -->
 <!-- The position of the TF frame has not been measured at all and needs to be calibrated. -->
-<robot name="robotiq_2f_85" xmlns:xacro="http://www.ros.org/wiki/xacro">
+<robot name="robotiq_2f_85"
+    xmlns:xacro="http://www.ros.org/wiki/xacro">
     <xacro:macro name="robotiq_2f_85" params="prefix parent">
         <!-- Spawn and attach robotiq 85 gripper -->
         <xacro:include filename="$(find robotiq_2f_85_gripper_visualization)/urdf/robotiq_arg2f_85_macro.xacro" />
-        <xacro:robotiq_arg2f_85 prefix="${prefix}" transmission_hw_interface="hardware_interface/EffortJointInterface" />
+        <xacro:robotiq_arg2f_85 prefix="${prefix}" transmission_hw_interface="hardware_interface/PositionJointInterface" />
         <joint name="robotiq_85_base_joint" type="fixed">
             <parent link="${parent}" />
             <child link="${prefix}robotiq_arg2f_base_link" />
-            <origin xyz="0.01 0 0" rpy="${pi} ${-pi/2} 0" /> <!-- This 0.01 offset is the Robotiq/UR coupling -->
+            <origin xyz="0.01 0 0" rpy="${pi} ${-pi/2} 0" />
+            <!-- This 0.01 offset is the Robotiq/UR coupling -->
         </joint>
         <!-- robotiq coupling link -->
@@ -37,58 +39,45 @@
         <!-- Mimic joints plugin-->
         <gazebo>
-            <plugin filename="libroboticsgroup_upatras_gazebo_mimic_joint_plugin.so" name="${prefix}mimic_robotiq_85_1">
-                <joint>${prefix}finger_joint</joint>
-                <mimicJoint>${prefix}left_inner_knuckle_joint</mimicJoint>
-                <multiplier>1.0</multiplier>
-            </plugin>
-            <plugin filename="libroboticsgroup_upatras_gazebo_mimic_joint_plugin.so" name="${prefix}mimic_robotiq_85_2">
-                <joint>${prefix}finger_joint</joint>
-                <mimicJoint>${prefix}left_inner_finger_joint</mimicJoint>
-                <multiplier>-1.0</multiplier>
-            </plugin>
-            <plugin filename="libroboticsgroup_upatras_gazebo_mimic_joint_plugin.so" name="${prefix}mimic_robotiq_85_3">
-                <joint>${prefix}finger_joint</joint>
-                <mimicJoint>${prefix}right_inner_knuckle_joint</mimicJoint>
-                <multiplier>1.0</multiplier>
-            </plugin>
-            <plugin filename="libroboticsgroup_upatras_gazebo_mimic_joint_plugin.so" name="${prefix}mimic_robotiq_85_4">
-                <joint>${prefix}finger_joint</joint>
-                <mimicJoint>${prefix}right_inner_finger_joint</mimicJoint>
-                <multiplier>-1.0</multiplier>
-            </plugin>
             <plugin filename="libroboticsgroup_upatras_gazebo_mimic_joint_plugin.so" name="${prefix}mimic_robotiq_85_5">
                 <joint>${prefix}finger_joint</joint>
                 <mimicJoint>${prefix}right_finger_joint</mimicJoint>
                 <multiplier>1.0</multiplier>
+                <hasPID/>
             </plugin>
         </gazebo>
+        <xacro:macro name="robotiq_2f_85_gazebo_link_properties" params="reference material">
+            <gazebo reference="${reference}">
+                <material>${material}</material>
+                <kp>1000000.0</kp>
+                <kd>1.0</kd>
+                <mu1>1.16</mu1>
+                <mu2>1.16</mu2>
+                <maxVel>0.0</maxVel>
+                <minDepth>0.001</minDepth>
+            </gazebo>
+        </xacro:macro>
         <!-- Links colors  -->
-        <gazebo reference="${prefix}robotiq_arg2f_base_link">
-            <material>Gazebo/Black</material>
-        </gazebo>
-        <gazebo reference="${prefix}left_outer_knuckle">
-            <material>Gazebo/Grey</material>
-        </gazebo>
-        <gazebo reference="${prefix}left_outer_finger">
-            <material>Gazebo/Black</material>
-        </gazebo>
-        <gazebo reference="${prefix}left_inner_finger">
-            <material>Gazebo/Grey</material>
-        </gazebo>
-        <gazebo reference="${prefix}left_inner_knuckle">
-            <material>Gazebo/Black</material>
-        </gazebo>
-        <gazebo reference="${prefix}right_outer_knuckle">
-            <material>Gazebo/Grey</material>
-        </gazebo>
-        <gazebo reference="${prefix}right_outer_finger">
-            <material>Gazebo/Black</material>
-        </gazebo>
-        <gazebo reference="${prefix}right_inner_finger">
-            <material>Gazebo/Grey</material>
-        </gazebo>
-        <gazebo reference="${prefix}right_inner_knuckle">
-            <material>Gazebo/Black</material>
-        </gazebo>
+        <xacro:robotiq_2f_85_gazebo_link_properties reference="${prefix}robotiq_arg2f_base_link" material="Gazebo/Black" />
+        <xacro:robotiq_2f_85_gazebo_link_properties reference="${prefix}left_outer_knuckle" material="Gazebo/Grey" />
+        <xacro:robotiq_2f_85_gazebo_link_properties reference="${prefix}left_outer_finger" material="Gazebo/Black" />
+        <xacro:robotiq_2f_85_gazebo_link_properties reference="${prefix}left_inner_finger" material="Gazebo/Grey" />
+        <xacro:robotiq_2f_85_gazebo_link_properties reference="${prefix}left_inner_knuckle" material="Gazebo/Black" />
+        <xacro:robotiq_2f_85_gazebo_link_properties reference="${prefix}right_outer_knuckle" material="Gazebo/Grey" />
+        <xacro:robotiq_2f_85_gazebo_link_properties reference="${prefix}right_outer_finger" material="Gazebo/Black" />
+        <xacro:robotiq_2f_85_gazebo_link_properties reference="${prefix}right_inner_finger" material="Gazebo/Grey" />
+        <xacro:robotiq_2f_85_gazebo_link_properties reference="${prefix}right_inner_knuckle" material="Gazebo/Black" />
+        <xacro:macro name="robotiq_2f_85_gazebo_joint_properties" params="reference">
+            <gazebo reference="${reference}">
+                <implicitSpringDamper>true</implicitSpringDamper>
+            </gazebo>
+        </xacro:macro>
+        <xacro:robotiq_2f_85_gazebo_joint_properties reference="${prefix}finger_joint"/>
+        <xacro:robotiq_2f_85_gazebo_joint_properties reference="${prefix}left_outer_finger_joint"/>
+        <xacro:robotiq_2f_85_gazebo_joint_properties reference="${prefix}left_inner_knuckle_joint"/>
+        <xacro:robotiq_2f_85_gazebo_joint_properties reference="${prefix}left_inner_finger_joint"/>
+        <xacro:robotiq_2f_85_gazebo_joint_properties reference="${prefix}right_finger_joint"/>
+        <xacro:robotiq_2f_85_gazebo_joint_properties reference="${prefix}right_outer_finger_joint"/>
+        <xacro:robotiq_2f_85_gazebo_joint_properties reference="${prefix}right_inner_knuckle_joint"/>
+        <xacro:robotiq_2f_85_gazebo_joint_properties reference="${prefix}right_inner_finger_joint"/>
     </xacro:macro>
 </robot>

File: homestri_robot_description/urdf/ur5e_macro.urdf.xacro (robot description, xacro)
@@ -8,9 +8,9 @@
     <xacro:ur_robot
       prefix="${prefix}"
-      joint_limits_parameters_file='$(find homestri_robot_description)/config/ur5e_joint_limits.yaml'
+      joint_limits_parameters_file='$(find homestri_robot_description)/config/gazebo_ur5e_joint_limits.yaml'
       kinematics_parameters_file='$(find ur_description)/config/ur5e/default_kinematics.yaml'
       physical_parameters_file='$(find ur_description)/config/ur5e/physical_parameters.yaml'
       visual_parameters_file='$(find ur_description)/config/ur5e/visual_parameters.yaml'
-      transmission_hw_interface='hardware_interface/EffortJointInterface'
+      transmission_hw_interface='hardware_interface/PositionJointInterface'
       safety_limits="false"
       safety_pos_margin="0.15"
@@ -38,26 +38,32 @@
       <origin rpy="0 0 0" xyz="0.163 0 0" />
     </joint>
-    <!-- Configure self collision properties per link -->
-    <gazebo reference="${prefix}shoulder_link">
-      <selfCollide>true</selfCollide>
-    </gazebo>
-    <gazebo reference="${prefix}upper_arm_link">
-      <selfCollide>true</selfCollide>
-    </gazebo>
-    <gazebo reference="${prefix}forearm_link">
-      <selfCollide>true</selfCollide>
-    </gazebo>
-    <gazebo reference="${prefix}wrist_1_link">
-      <selfCollide>true</selfCollide>
-    </gazebo>
-    <gazebo reference="${prefix}wrist_3_link">
-      <selfCollide>true</selfCollide>
-    </gazebo>
-    <gazebo reference="${prefix}wrist_2_link">
-      <selfCollide>true</selfCollide>
-    </gazebo>
-    <gazebo reference="${prefix}ee_link">
-      <selfCollide>true</selfCollide>
-    </gazebo>
+    <xacro:macro name="ur5e_gazebo_link_properties" params="reference">
+      <gazebo reference="${reference}">
+        <kp>1000000.0</kp>
+        <kd>1.0</kd>
+        <mu1>0.8</mu1>
+        <mu2>0.8</mu2>
+        <maxVel>0.0</maxVel>
+        <minDepth>0.001</minDepth>
+        <selfCollide>true</selfCollide>
+      </gazebo>
+    </xacro:macro>
+    <xacro:ur5e_gazebo_link_properties reference="${prefix}shoulder_link" />
+    <xacro:ur5e_gazebo_link_properties reference="${prefix}upper_arm_link" />
+    <xacro:ur5e_gazebo_link_properties reference="${prefix}forearm_link" />
+    <xacro:ur5e_gazebo_link_properties reference="${prefix}wrist_1_link" />
+    <xacro:ur5e_gazebo_link_properties reference="${prefix}wrist_2_link" />
+    <xacro:ur5e_gazebo_link_properties reference="${prefix}wrist_3_link" />
+    <xacro:macro name="ur5e_gazebo_joint_properties" params="reference">
+      <gazebo reference="${reference}">
+        <implicitSpringDamper>true</implicitSpringDamper>
+      </gazebo>
+    </xacro:macro>
+    <xacro:ur5e_gazebo_link_properties reference="${prefix}shoulder_pan_joint" />
+    <xacro:ur5e_gazebo_link_properties reference="${prefix}shoulder_lift_joint" />
+    <xacro:ur5e_gazebo_link_properties reference="${prefix}elbow_joint" />
+    <xacro:ur5e_gazebo_link_properties reference="${prefix}wrist_1_joint" />
+    <xacro:ur5e_gazebo_link_properties reference="${prefix}wrist_2_joint" />
+    <xacro:ur5e_gazebo_link_properties reference="${prefix}wrist_3_joint" />
   </xacro:macro>
 </robot>

Commit message: cleanup and reorganize code, added BT and manip action server code

File: homestri_moveit_config/config/gazebo_base_scene.urdf (robot description, URDF)
Before this commit: robot base_scene, 26 links, 25 joints
Links:
- removed link coupling
- added link robotiq_85_coupling, mass 0.1; collision cylinder length=0.01 radius=0.0375; visual cylinder length=0.01 radius=0.0375
- link left_inner_finger: mass 0.01957844415989899 -> 0.05873533247969697
- link left_inner_finger_pad: mass 0.014144625000000003 -> 0.04243387500000001
- link left_inner_knuckle: mass 0.029949543712543904 -> 0.08984863113763171
- link left_outer_finger: mass 0.02729659380694228 -> 0.08188978142082684
- link left_outer_knuckle: mass 0.018476648450763997 -> 0.055429945352291995
- link right_inner_finger: mass 0.01957844415989899 -> 0.05873533247969697
- link right_inner_finger_pad: mass 0.014144625000000003 -> 0.04243387500000001
- link right_inner_knuckle: mass 0.029949543712543904 -> 0.08984863113763171
- link right_outer_finger: mass 0.02729659380694228 -> 0.08188978142082684
- link right_outer_knuckle: mass 0.018476648450763997 -> 0.055429945352291995
Joints:
- removed joint coupling_joint
- removed joint world_joint
- added joint robotiq_85_coupling_joint: type fixed, parent ee_link, child robotiq_85_coupling, origin xyz=0 0 0 rpy=0 0 0
- added joint ur5e_base_joint: type fixed, parent world, child base_link, origin xyz=0 0 0 rpy=0 0 0
- joint finger_joint: limit lower=0 upper=0.8 effort=1000 velocity=0.5 -> lower=0 upper=0.8 effort=100.0 velocity=2.0
- joint left_inner_finger_joint: limit lower=-0.8757 upper=0 effort=1000 velocity=0.5 -> lower=-0.8757 upper=0 effort=100.0 velocity=2.0
- joint left_inner_knuckle_joint: limit lower=0 upper=0.8757 effort=1000 velocity=0.5 -> lower=0 upper=0.8757 effort=100.0 velocity=2.0
- joint right_finger_joint: limit lower=0 upper=0.81 effort=1000 velocity=0.5 -> lower=0 upper=0.81 effort=100.0 velocity=2.0
- joint right_inner_finger_joint: limit lower=-0.8757 upper=0 effort=1000 velocity=0.5 -> lower=-0.8757 upper=0 effort=100.0 velocity=2.0
- joint right_inner_knuckle_joint: limit lower=0 upper=0.8757 effort=1000 velocity=0.5 -> lower=0 upper=0.8757 effort=100.0 velocity=2.0
- joint robotiq_85_base_joint: parent ee_link -> robotiq_85_coupling

File: homestri_robot_description/urdf/base_scene.urdf.xacro (robot description, xacro)
@@ -1,20 +1,22 @@
 <?xml version="1.0"?>
-<robot xmlns:xacro="http://www.ros.org/wiki/xacro"
-       name="base_scene" >
-  <!-- ur5e arm and robotiq gripper -->
-  <xacro:include filename="$(find homestri_robot_description)/urdf/ur5e_macro.urdf.xacro" />
-  <xacro:ur5e prefix="" />
-  <xacro:include filename="$(find homestri_robot_description)/urdf/robotiq_2f_85_macro.urdf.xacro" />
-  <xacro:robotiq_2f_85 prefix="" parent="ee_link" />
-  <!-- scene environment (pedestal and table) -->
-  <!-- <xacro:include filename="$(find homestri_robot_description)/urdf/environment.urdf.xacro" />
-  <xacro:environment /> -->
-  <!-- attach table to world. -->
+<robot xmlns:xacro="http://www.ros.org/wiki/xacro" name="base_scene">
+  <xacro:include filename="$(find homestri_robot_description)/urdf/ur5e_macro.xacro" />
+  <xacro:include filename="$(find homestri_robot_description)/urdf/robotiq_2f_85_macro.xacro" />
+  <xacro:ur5e
+    prefix=""
+    parent="world"
+    transmission_hw_interface="hardware_interface/PositionJointInterface"
+  >
+    <origin xyz="0 0 0" rpy="0 0 0" />
+  </xacro:ur5e>
+  <xacro:robotiq_2f_85
+    prefix=""
+    parent="ee_link"
+    transmission_hw_interface="hardware_interface/PositionJointInterface"
+    coupling_width="0.01"
+  >
+    <origin xyz="0 0 0" rpy="0 0 0" />
+  </xacro:robotiq_2f_85>
   <link name="world" />
-  <joint name="world_joint" type="fixed">
-    <parent link="world" />
-    <child link="base_link" />
-    <origin xyz="0 0 0" rpy="0 0 0" />
-  </joint>
   <gazebo>
     <plugin name="ros_control" filename="libgazebo_ros_control.so">

File: homestri_robot_description/urdf/ur5e_macro.xacro (robot description, xacro)
@@ -3,5 +3,5 @@
 <!-- The position of the TF frame has not been measured at all and needs to be calibrated. -->
 <robot name="ur5e" xmlns:xacro="http://www.ros.org/wiki/xacro">
-  <xacro:macro name="ur5e" params="prefix">
+  <xacro:macro name="ur5e" params="prefix parent transmission_hw_interface *origin">
     <!-- ur5e -->
     <xacro:include filename="$(find ur_description)/urdf/inc/ur_macro.xacro" />
@@ -12,9 +12,14 @@
       physical_parameters_file='$(find ur_description)/config/ur5e/physical_parameters.yaml'
       visual_parameters_file='$(find ur_description)/config/ur5e/visual_parameters.yaml'
-      transmission_hw_interface='hardware_interface/PositionJointInterface'
+      transmission_hw_interface="${transmission_hw_interface}"
       safety_limits="false"
       safety_pos_margin="0.15"
       safety_k_position="20"
     />
+    <joint name="${prefix}ur5e_base_joint" type="fixed">
+      <parent link="${parent}" />
+      <child link="${prefix}base_link" />
+      <xacro:insert_block name="origin" />
+    </joint>
     <!-- end effector link -->
     <link name="${prefix}ee_link">
@@ -38,4 +43,5 @@
       <origin rpy="0 0 0" xyz="0.163 0 0" />
     </joint>
+    <!-- ############ GAZEBO PROPERTIES ############ -->
     <xacro:macro name="ur5e_gazebo_link_properties" params="reference">
       <gazebo reference="${reference}">

File: homestri_scene_description/urdf/plastic_bin.urdf (robot description, URDF)
Before this commit: robot plastic_bin, 1 links, 0 joints
Links:
- link base_link: geometry collision mesh filename=package://homestri_scene_description/meshes/plastic_bin.stl scale=0.001 0.001 0.001; visual mesh filename=package://homestri_scene_description/meshes/plastic_bin.stl scale=0.001 0.001 0.001

Commit message: updated moveit_config and added simple pedestal and ground

File: homestri_moveit_config/config/gazebo_base_scene.urdf (robot description, URDF)
Before this commit: robot base_scene, 26 links, 25 joints
Links:
- added link ground, mass 0.1; collision box size=5 5 0.02
- added link pedestal, mass .006784; collision cylinder length=0.2 radius=0.12; visual cylinder length=0.2 radius=0.12
Joints:
- added joint ground_to_world: type fixed, parent world, child ground, origin xyz=0 0 0
- added joint pedestal_to_ground: type fixed, parent ground, child pedestal, origin xyz=0 0 0.2
- joint ur5e_base_joint: parent world -> pedestal

File: homestri_robot_description/urdf/base_scene.xacro (robot description, xacro)
@@ -1,9 +1,14 @@
 <?xml version="1.0"?>
 <robot xmlns:xacro="http://www.ros.org/wiki/xacro" name="base_scene">
+  <xacro:include filename="$(find homestri_robot_description)/urdf/environment.xacro" />
   <xacro:include filename="$(find homestri_robot_description)/urdf/ur5e_macro.xacro" />
   <xacro:include filename="$(find homestri_robot_description)/urdf/robotiq_2f_85_macro.xacro" />
+  <xacro:environment
+    pedestal_height="0.2"
+    pedestal_radius="0.12"
+  />
   <xacro:ur5e
     prefix=""
-    parent="world"
+    parent="pedestal"
     transmission_hw_interface="hardware_interface/PositionJointInterface"
   >

File: homestri_robot_description/urdf/robotiq_2f_85_macro.xacro (robot description, xacro)
@@ -58,4 +58,5 @@
     </xacro:macro>
     <!-- Links colors  -->
+    <xacro:robotiq_2f_85_gazebo_link_properties reference="${prefix}robotiq_85_coupling" material="Gazebo/Black" />
     <xacro:robotiq_2f_85_gazebo_link_properties reference="${prefix}robotiq_arg2f_base_link" material="Gazebo/Black" />
     <xacro:robotiq_2f_85_gazebo_link_properties reference="${prefix}left_outer_knuckle" material="Gazebo/Grey" />
