Commit message: updated urdf for new gripper coupler

File: homestri_moveit_config/config/gazebo_base_scene.urdf (robot description, URDF)
Before this commit: robot base_scene, 28 links, 27 joints
Links:
- removed link pedestal
- removed link robotiq_85_coupling
- removed link robotiq_arg2f_base_link
- added link cable_protector, mass 0.03136596181658943; collision mesh filename=package://robotiq_2f_85_gripper_description/meshes/collisio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 scale=0.001 0.001 0.001; visual mesh filename=package://robotiq_2f_85_gripper_description/meshes/visual/r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 scale=0.001 0.001 0.001
- added link coupler, mass 0.10117556100473797; collision mesh filename=package://robotiq_2f_85_gripper_description/meshes/collisio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 scale=0.001 0.001 0.001; visual mesh filename=package://robotiq_2f_85_gripper_description/meshes/visual/r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 scale=0.001 0.001 0.001
- added link gripper_body, mass 0.22651999999800307; collision mesh filename=package://robotiq_2f_85_gripper_description/meshes/collisio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; visual mesh filename=package://robotiq_2f_85_gripper_description/meshes/visual/r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
- link left_inner_finger: geometry collision mesh filename=package://robotiq_2f_85_gripper_description/meshes/collisio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 scale=0.001 0.001 0.001; visual mesh filename=package://robotiq_2f_85_gripper_description/meshes/visual/r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 scale=0.001 0.001 0.001
- link left_inner_knuckle: geometry collision mesh filename=package://robotiq_2f_85_gripper_description/meshes/collisio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 scale=0.001 0.001 0.001; visual mesh filename=package://robotiq_2f_85_gripper_description/meshes/visual/r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 scale=0.001 0.001 0.001
- link left_outer_finger: geometry collision mesh filename=package://robotiq_2f_85_gripper_description/meshes/collisio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 scale=0.001 0.001 0.001; visual mesh filename=package://robotiq_2f_85_gripper_description/meshes/visual/r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 scale=0.001 0.001 0.001
- link left_outer_knuckle: geometry collision mesh filename=package://robotiq_2f_85_gripper_description/meshes/collisio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 scale=0.001 0.001 0.001; visual mesh filename=package://robotiq_2f_85_gripper_description/meshes/visual/r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 scale=0.001 0.001 0.001
- link right_inner_finger: geometry collision mesh filename=package://robotiq_2f_85_gripper_description/meshes/collisio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 scale=0.001 0.001 0.001; visual mesh filename=package://robotiq_2f_85_gripper_description/meshes/visual/r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 scale=0.001 0.001 0.001
- link right_inner_knuckle: geometry collision mesh filename=package://robotiq_2f_85_gripper_description/meshes/collisio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 scale=0.001 0.001 0.001; visual mesh filename=package://robotiq_2f_85_gripper_description/meshes/visual/r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 scale=0.001 0.001 0.001
- link right_outer_finger: geometry collision mesh filename=package://robotiq_2f_85_gripper_description/meshes/collisio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 scale=0.001 0.001 0.001; visual mesh filename=package://robotiq_2f_85_gripper_description/meshes/visual/r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 scale=0.001 0.001 0.001
- link right_outer_knuckle: geometry collision mesh filename=package://robotiq_2f_85_gripper_description/meshes/collisio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 scale=0.001 0.001 0.001; visual mesh filename=package://robotiq_2f_85_gripper_description/meshes/visual/r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 scale=0.001 0.001 0.001
Joints:
- removed joint pedestal_to_ground
- removed joint robotiq_85_base_joint
- removed joint robotiq_85_coupling_joint
- added joint cable_protector_joint: type fixed, parent coupler, child cable_protector, origin xyz=-0.0105 0.034 0.002999999999999999 rpy=0 0 0
- added joint coupler_joint: type fixed, parent ee_link, child coupler, origin xyz=0 0 0 rpy=-1.5707963267948966 3.141592653589793 -1.5707963267948966
- added joint gripper_body_joint: type fixed, parent coupler, child gripper_body, origin xyz=0 0 0.011 rpy=0 0 -1.5707963267948966
- joint finger_joint: parent robotiq_arg2f_base_link -> gripper_body
- joint left_inner_knuckle_joint: parent robotiq_arg2f_base_link -> gripper_body
- joint right_finger_joint: parent robotiq_arg2f_base_link -> gripper_body
- joint right_inner_knuckle_joint: parent robotiq_arg2f_base_link -> gripper_body
- joint ur5e_base_joint: parent pedestal -> world

File: homestri_robot_description/urdf/base_scene.xacro (robot description, xacro)
@@ -3,5 +3,5 @@
   <xacro:include filename="$(find homestri_robot_description)/urdf/workspace.xacro" />
   <xacro:include filename="$(find homestri_robot_description)/urdf/ur5e_macro.xacro" />
-  <xacro:include filename="$(find homestri_robot_description)/urdf/robotiq_2f_85_macro.xacro" />
+  <xacro:include filename="$(find robotiq_2f_85_gripper_description)/urdf/robotiq_arg2f_85_macro.xacro" />
   <xacro:workspace />
   <xacro:ur5e
@@ -12,12 +12,11 @@
     <origin xyz="0 0 0" rpy="0 0 0" />
   </xacro:ur5e>
-  <xacro:robotiq_2f_85
+  <xacro:robotiq_arg2f_85
     prefix=""
     parent="ee_link"
     transmission_hw_interface="hardware_interface/PositionJointInterface"
-    coupling_width="0.01"
   >
-    <origin xyz="0 0 0" rpy="0 0 0" />
-  </xacro:robotiq_2f_85>
+    <origin xyz="0 0 0" rpy="${-pi/2} ${pi} ${-pi/2}" />
+  </xacro:robotiq_arg2f_85 >
   <link name="world" />
   <gazebo>
