Commit message: update b_bot with table and pedestal

File: homestri_description/urdf/scenes/b_bot_scene.xacro (robot description, xacro)
@@ -7,5 +7,5 @@
     <xacro:ur5e
         prefix=""
-        parent="world"
+        parent="pedestal"
         transmission_hw_interface="hardware_interface/PositionJointInterface"
     >

File: homestri_description/urdf/workspaces/b_bot_workspace.xacro (robot description, xacro)
@@ -4,21 +4,21 @@
 <robot name="b_bot_workspace" xmlns:xacro="http://www.ros.org/wiki/xacro">
   <xacro:macro name="b_bot_workspace">
-  <!-- <xacro:macro name="workspace" params="pedestal_height:=0.2 pedestal_radius:=0.2"> -->
-    <!-- <link name="pedestal">
+    <!-- <xacro:macro name="workspace" params="pedestal_height:=0.2 pedestal_radius:=0.2"> -->
+    <link name="pedestal">
+      <collision>
+        <origin xyz="0 0 -0.2" rpy="0 0 0" />
+        <geometry>
+          <box size="0.2 0.2 0.4" />
+        </geometry>
+      </collision>
       <visual>
-        <origin rpy="0 0 0" xyz="0 0 ${-pedestal_height/2}"/>
+        <origin xyz="0 0 -0.2" rpy="0 0 0" />
         <geometry>
-          <cylinder length="${pedestal_height}" radius="${pedestal_radius}"/>
+          <box size="0.2 0.2 0.4" />
         </geometry>
         <material name="grey">
-            <color rgba=".5 .5 .5 1"/>
+          <color rgba=".5 .5 .5 1.0" />
         </material>
       </visual>
-      <collision>
-        <origin rpy="0 0 0" xyz="0 0 ${-pedestal_height/2}"/>
-        <geometry>
-          <cylinder length="${pedestal_height}" radius="${pedestal_radius}"/>
-        </geometry>
-      </collision>
       <inertial>
         <origin xyz="0.0 0.0 0.02" rpy="0 0 0" />
@@ -26,12 +26,34 @@
         <inertia ixx=".18e-05" iyy=".18e-05" izz=".18e-05" ixy="0.0" iyz="0.0" ixz="0.0" />
       </inertial>
-    </link> -->
+    </link>
+    <link name="table">
+      <collision>
+        <origin xyz="0 0 .25" rpy="0 0 0" />
+        <geometry>
+          <box size="1 1 0.5" />
+        </geometry>
+      </collision>
+      <visual>
+        <origin xyz="0 0 .25" rpy="0 0 0" />
+        <geometry>
+          <box size="1 1 0.5" />
+        </geometry>
+        <material name="grey">
+          <color rgba=".5 .5 .5 1.0" />
+        </material>
+      </visual>
+      <inertial>
+        <origin xyz="0.0 0.0 0.02" rpy="0 0 0" />
+        <mass value=".006784" />
+        <inertia ixx=".18e-05" iyy=".18e-05" izz=".18e-05" ixy="0.0" iyz="0.0" ixz="0.0" />
+      </inertial>
+    </link>
     <link name="ground">
-        <collision>
-            <origin rpy="0 0 0" xyz="0 0 -0.01"/>
-            <geometry>
-                <box size="5 5 0.02" />
-            </geometry>
-        </collision>
+      <collision>
+        <origin rpy="0 0 0" xyz="0 0 -0.01" />
+        <geometry>
+          <box size="5 5 0.02" />
+        </geometry>
+      </collision>
     </link>
     <!-- <joint name="pedestal_to_world" type="fixed">
@@ -41,10 +63,20 @@
     </joint> -->
     <joint name="ground_to_world" type="fixed">
-        <parent link="world"/>
-        <child link="ground"/>
-        <origin xyz="0 0 0" />
+      <parent link="world" />
+      <child link="ground" />
+      <origin xyz="0 0 0" />
+    </joint>
+    <joint name="table_to_world" type="fixed">
+      <parent link="world" />
+      <child link="table" />
+      <origin xyz="1 0 0" />
+    </joint>
+    <joint name="pedestal_to_world" type="fixed">
+      <parent link="world" />
+      <child link="pedestal" />
+      <origin xyz="0 0 0.4" />
     </joint>
     <gazebo reference="pedestal">
-        <material>Gazebo/Grey</material>
+      <material>Gazebo/Grey</material>
     </gazebo>
   </xacro:macro>

Commit message: added camera to b_bot description

File: homestri_description/urdf/scenes/b_bot_scene.xacro (robot description, xacro)
@@ -3,5 +3,6 @@
     <xacro:include filename="$(find homestri_description)/urdf/workspaces/b_bot_workspace.xacro" />
     <xacro:include filename="$(find homestri_description)/urdf/macros/ur5e_macro.xacro" />
-    <xacro:include filename="$(find onrobot_rg2ft_description)/urdf/onrobot_rg2ft_macro.xacro" />
+    <xacro:include
+        filename="$(find homestri_description)/urdf/macros/onrobot_realsense_macro.xacro" />
     <xacro:b_bot_workspace />
     <xacro:ur5e
@@ -13,11 +14,11 @@
         <origin xyz="0 0 0" rpy="0 0 0" />
     </xacro:ur5e>
-    <xacro:onrobot_rg2ft
+    <xacro:onrobot_realsense
         prefix=""
         parent="ee_link"
-        hw_interface="hardware_interface/PositionJointInterface"
+        transmission_hw_interface="hardware_interface/PositionJointInterface"
     >
-        <origin xyz="0 0 0" rpy="${pi/2} ${0} ${pi/2}" />
-    </xacro:onrobot_rg2ft>
+        <origin xyz="0 0 0" rpy="${-pi/2} ${0} ${-pi/2}" />
+    </xacro:onrobot_realsense>
     <link name="world" />
     <gazebo>
