Commit message: add realsense mount to urdf

File: homestri_description/urdf/scenes/a_bot_scene.xacro (robot description, xacro)
@@ -4,5 +4,5 @@
     <xacro:include filename="$(find homestri_description)/urdf/macros/ur5e_macro.xacro" />
     <xacro:include
-        filename="$(find robotiq_2f_85_gripper_description)/urdf/robotiq_arg2f_85_macro.xacro" />
+        filename="$(find homestri_description)/urdf/macros/robotiq_realsense_macro.xacro" />
     <xacro:a_bot_workspace />
     <xacro:ur5e
@@ -14,11 +14,11 @@
         <origin xyz="0 0 0" rpy="0 0 0" />
     </xacro:ur5e>
-    <xacro:robotiq_arg2f_85
+    <xacro:robotiq_realsense
         prefix=""
         parent="ee_link"
         transmission_hw_interface="hardware_interface/PositionJointInterface"
     >
-        <origin xyz="0 0 0" rpy="${-pi/2} ${pi} ${-pi/2}" />
-    </xacro:robotiq_arg2f_85>
+        <origin xyz="0 0 0" rpy="${-pi/2} ${0} ${-pi/2}" />
+    </xacro:robotiq_realsense>
     <link name="world" />
     <gazebo>

Commit message: added assembly to a_bot scene

File: homestri_description/urdf/scenes/a_bot_scene.xacro (robot description, xacro)
@@ -5,8 +5,14 @@
     <xacro:include
         filename="$(find homestri_description)/urdf/macros/robotiq_realsense_macro.xacro" />
-    <xacro:a_bot_workspace />
+    <xacro:a_bot_workspace
+        pedestal_height="0.6"
+        pedestal_radius="0.15"
+        table_height="0.4"
+        table_y="-0.8"
+        table_x="0.25"
+    />
     <xacro:ur5e
         prefix=""
-        parent="world"
+        parent="pedestal"
         gripper_tip_offset="0.163"
         transmission_hw_interface="hardware_interface/PositionJointInterface"

File: homestri_description/urdf/workspaces/a_bot_workspace.xacro (robot description, xacro)
@@ -1,22 +1,74 @@
 <?xml version="1.0"?>
-<!-- This macro adds a convenient TF frame at the tip of the closed gripper. -->
-<!-- The position of the TF frame has not been measured at all and needs to be calibrated. -->
 <robot name="a_bot_workspace" xmlns:xacro="http://www.ros.org/wiki/xacro">
-  <xacro:macro name="a_bot_workspace">
-  <!-- <xacro:macro name="workspace" params="pedestal_height:=0.2 pedestal_radius:=0.2"> -->
-    <!-- <link name="pedestal">
+  <xacro:macro name="a_bot_workspace"
+    params="pedestal_height:=0.2 pedestal_radius:=0.2 table_height:=0.2 table_y:=0.5 table_x:=0.5">
+    <link name="static_assembly">
+      <inertial>
+        <origin xyz="-0.0019215269775362533 0.02238591812637603 0.00014773610274437554"
+          rpy="0 0 0" />
+        <mass value="0.0478036670662668" />
+        <inertia ixx="4.3e-05" iyy="2.2e-05" izz="6.4e-05" ixy="3e-06" iyz="1e-06" ixz="0.0" />
+      </inertial>
       <visual>
-        <origin rpy="0 0 0" xyz="0 0 ${-pedestal_height/2}"/>
+        <origin xyz="0 0 0" rpy="0 0 ${pi}" />
         <geometry>
-          <cylinder length="${pedestal_height}" radius="${pedestal_radius}"/>
+          <mesh
+            filename="package://homestri_description/meshes/components/visual/2assembly_nonmoving_components.stl"
+            scale="0.001 0.001 0.001" />
         </geometry>
-        <material name="grey">
-            <color rgba=".5 .5 .5 1"/>
+        <material name="">
+          <color rgba="${153/255} ${255/255} ${153/255} 1" />
         </material>
       </visual>
       <collision>
-        <origin rpy="0 0 0" xyz="0 0 ${-pedestal_height/2}"/>
+        <origin xyz="0 0 0" rpy="0 0 ${pi}" />
         <geometry>
-          <cylinder length="${pedestal_height}" radius="${pedestal_radius}"/>
+          <mesh
+            filename="package://homestri_description/meshes/components/collision/2assembly_nonmoving_components.stl"
+            scale="0.001 0.001 0.001" />
+        </geometry>
+      </collision>
+    </link>
+    <link name="moving_assembly">
+      <inertial>
+        <origin xyz="-0.0019215269775362533 0.02238591812637603 0.00014773610274437554"
+          rpy="0 0 0" />
+        <mass value="0.0478036670662668" />
+        <inertia ixx="4.3e-05" iyy="2.2e-05" izz="6.4e-05" ixy="3e-06" iyz="1e-06" ixz="0.0" />
+      </inertial>
+      <visual>
+        <origin xyz="0 0 0" rpy="0 0 ${pi}" />
+        <geometry>
+          <mesh
+            filename="package://homestri_description/meshes/components/visual/1assembly_moving_components.stl"
+            scale="0.001 0.001 0.001" />
+        </geometry>
+        <material name="">
+          <color rgba="${255/255} ${153/255} ${255/255} 1" />
+        </material>
+      </visual>
+      <collision>
+        <origin xyz="0 0 0" rpy="0 0 ${pi}" />
+        <geometry>
+          <mesh
+            filename="package://homestri_description/meshes/components/collision/1assembly_moving_components.stl"
+            scale="0.001 0.001 0.001" />
+        </geometry>
+      </collision>
+    </link>
+    <link name="pedestal">
+      <visual>
+        <origin rpy="0 0 0" xyz="0 0 ${-pedestal_height/2}" />
+        <geometry>
+          <cylinder length="${pedestal_height}" radius="${pedestal_radius}" />
+        </geometry>
+        <material name="grey">
+          <color rgba=".5 .5 .5 1" />
+        </material>
+      </visual>
+      <collision>
+        <origin rpy="0 0 0" xyz="0 0 ${-pedestal_height/2}" />
+        <geometry>
+          <cylinder length="${pedestal_height}" radius="${pedestal_radius}" />
         </geometry>
       </collision>
@@ -26,25 +78,51 @@
         <inertia ixx=".18e-05" iyy=".18e-05" izz=".18e-05" ixy="0.0" iyz="0.0" ixz="0.0" />
       </inertial>
-    </link> -->
-    <link name="ground">
-        <collision>
-            <origin rpy="0 0 0" xyz="0 0 -0.01"/>
-            <geometry>
-                <box size="5 5 0.02" />
-            </geometry>
-        </collision>
     </link>
-    <!-- <joint name="pedestal_to_world" type="fixed">
-        <parent link="world"/>
-        <child link="pedestal"/>
-        <origin xyz="0 0 ${pedestal_height}" />
-    </joint> -->
-    <joint name="ground_to_world" type="fixed">
-        <parent link="world"/>
-        <child link="ground"/>
-        <origin xyz="0 0 0" />
+    <link name="table">
+      <collision>
+        <origin xyz="0 -0.31 ${-table_height/2}" rpy="0 0 0" />
+        <geometry>
+          <box size="1 0.62 ${table_height}" />
+        </geometry>
+      </collision>
+      <visual>
+        <origin xyz="0 -0.31 ${-table_height/2}" rpy="0 0 0" />
+        <geometry>
+          <box size="1 0.62 ${table_height}" />
+        </geometry>
+        <material name="grey">
+          <color rgba=".5 .5 .5 1.0" />
+        </material>
+      </visual>
+      <inertial>
+        <origin xyz="0.0 0.0 0.3" rpy="0 0 0" />
+        <mass value=".006784" />
+        <inertia ixx=".18e-05" iyy=".18e-05" izz=".18e-05" ixy="0.0" iyz="0.0" ixz="0.0" />
+      </inertial>
+    </link>
+    <joint name="static_assembly_to_table" type="fixed">
+      <parent link="table" />
+      <child link="static_assembly" />
+      <origin xyz="0 -.0245 0" />
+    </joint>
+    <joint name="moving_assembly_joint" type="prismatic">
+      <axis xyz="0 -1 0"/>
+      <parent link="static_assembly" />
+      <child link="moving_assembly" />
+      <limit effort="1000.0" lower="0" upper=".38" velocity="0.5"/>
+      <origin rpy="0 0 0" xyz="0 0 0"/>
+    </joint>
+    <joint name="table_to_world" type="fixed">
+      <parent link="world" />
+      <child link="table" />
+      <origin xyz="${table_x} ${table_y} ${table_height}" />
+    </joint>
+    <joint name="pedestal_to_world" type="fixed">
+      <parent link="world" />
+      <child link="pedestal" />
+      <origin xyz="0 0 ${pedestal_height}" />
     </joint>
     <gazebo reference="pedestal">
-        <material>Gazebo/Grey</material>
+      <material>Gazebo/Grey</material>
     </gazebo>
   </xacro:macro>
