Commit message: almost working demo

File: homestri_b_bot_moveit_config/config/gazebo_b_bot_scene.urdf (robot description, URDF)
Before this commit: robot b_bot_scene, 24 links, 23 joints
Links:
- added link closet, mass .006784; collision box size=4 2 2
- added link pedestal, mass .006784; collision box size=0.35 0.35 0.814; visual box size=0.35 0.35 0.814
- added link table, mass .006784; collision box size=1 2 0.917; visual box size=1 2 0.917
Joints:
- added joint closet_to_world: type fixed, parent world, child closet, origin xyz=1.45 1.45 0
- added joint pedestal_to_world: type fixed, parent world, child pedestal, origin xyz=0 0 0.814
- added joint table_to_world: type fixed, parent world, child table, origin xyz=-1.37 0 0
- joint shoulder_pan_joint: limit lower=-3.141592653589793 upper=3.141592653589793 effort=150.0 velocity=3.141592653589793 -> lower=-6.283185307179586 upper=6.283185307179586 effort=150.0 velocity=3.141592653589793
- joint ur5e_base_joint: parent world -> pedestal

File: homestri_description/urdf/macros/ur5e_macro.xacro (robot description, xacro)
@@ -3,5 +3,5 @@
 <!-- The position of the TF frame has not been measured at all and needs to be calibrated. -->
 <robot name="ur5e" xmlns:xacro="http://www.ros.org/wiki/xacro">
-  <xacro:macro name="ur5e" params="prefix parent transmission_hw_interface *origin">
+  <xacro:macro name="ur5e" params="prefix parent transmission_hw_interface gripper_tip_offset *origin">
     <!-- ur5e -->
     <xacro:include filename="$(find ur_description)/urdf/inc/ur_macro.xacro" />
@@ -41,5 +41,5 @@
       <parent link="${prefix}ee_link" />
       <child link="${prefix}gripper_tip_link" />
-      <origin rpy="0 0 0" xyz="0.163 0 0" />
+      <origin rpy="0 0 0" xyz="${gripper_tip_offset} 0 0" />
     </joint>
     <!-- ############ GAZEBO PROPERTIES ############ -->

File: homestri_description/urdf/scenes/a_bot_scene.xacro (robot description, xacro)
@@ -9,4 +9,5 @@
         prefix=""
         parent="world"
+        gripper_tip_offset="0.163"
         transmission_hw_interface="hardware_interface/PositionJointInterface"
     >

File: homestri_description/urdf/scenes/b_bot_scene.xacro (robot description, xacro)
@@ -8,4 +8,5 @@
         prefix=""
         parent="pedestal"
+        gripper_tip_offset="0.223"
         transmission_hw_interface="hardware_interface/PositionJointInterface"
     >

File: homestri_description/urdf/workspaces/b_bot_workspace.xacro (robot description, xacro)
@@ -7,13 +7,13 @@
     <link name="pedestal">
       <collision>
-        <origin xyz="0 0 -0.2" rpy="0 0 0" />
+        <origin xyz="0 0 -0.407" rpy="0 0 0" />
         <geometry>
-          <box size="0.2 0.2 0.4" />
+          <box size="0.35 0.35 0.814" />
         </geometry>
       </collision>
       <visual>
-        <origin xyz="0 0 -0.2" rpy="0 0 0" />
+        <origin xyz="0 0 -0.407" rpy="0 0 0" />
         <geometry>
-          <box size="0.2 0.2 0.4" />
+          <box size="0.35 0.35 0.814" />
         </geometry>
         <material name="grey">
@@ -29,13 +29,13 @@
     <link name="table">
       <collision>
-        <origin xyz="0 0 .3" rpy="0 0 0" />
+        <origin xyz="0 0 0.4585" rpy="0 0 0" />
         <geometry>
-          <box size="1 1 0.6" />
+          <box size="1 2 0.917" />
         </geometry>
       </collision>
       <visual>
-        <origin xyz="0 0 .3" rpy="0 0 0" />
+        <origin xyz="0 0 0.4585" rpy="0 0 0" />
         <geometry>
-          <box size="1 1 0.6" />
+          <box size="1 2 0.917" />
         </geometry>
         <material name="grey">
@@ -48,4 +48,37 @@
         <inertia ixx=".18e-05" iyy=".18e-05" izz=".18e-05" ixy="0.0" iyz="0.0" ixz="0.0" />
       </inertial>
+    </link>
+    <link name="wall_1">
+      <collision>
+        <origin rpy="0 ${pi/2} 0" xyz="-0.45 0 0" />
+        <geometry>
+          <box size="5 5 0.02" />
+        </geometry>
+        <material name="grey">
+          <color rgba=".5 .5 .5 1.0" />
+        </material>
+      </collision>
+    </link>
+    <link name="wall_2">
+      <collision>
+        <origin rpy="${pi/2} 0 0" xyz="0 -0.4 0" />
+        <geometry>
+          <box size="5 5 0.02" />
+        </geometry>
+        <material name="grey">
+          <color rgba=".5 .5 .5 1.0" />
+        </material>
+      </collision>
+    </link>
+    <link name="wall_3">
+      <collision>
+        <origin rpy="0 0 0" xyz="0 0 1.7" />
+        <geometry>
+          <box size="5 5 0.02" />
+        </geometry>
+        <material name="grey">
+          <color rgba=".5 .5 .5 1.0" />
+        </material>
+      </collision>
     </link>
     <link name="ground">
@@ -65,10 +98,25 @@
       <parent link="world" />
       <child link="table" />
-      <origin xyz="0 -1 0" />
+      <origin xyz="1.37 0 0" />
+    </joint>
+    <joint name="wall_1_to_world" type="fixed">
+      <parent link="world" />
+      <child link="wall_1" />
+      <origin xyz="0 0 0" />
+    </joint>
+    <joint name="wall_2_to_world" type="fixed">
+      <parent link="world" />
+      <child link="wall_2" />
+      <origin xyz="0 0 0" />
+    </joint>
+    <joint name="wall_3_to_world" type="fixed">
+      <parent link="world" />
+      <child link="wall_3" />
+      <origin xyz="0 0 0" />
     </joint>
     <joint name="pedestal_to_world" type="fixed">
       <parent link="world" />
       <child link="pedestal" />
-      <origin xyz="0 0 0.4" />
+      <origin xyz="0 0 0.814" rpy="0 0 ${pi/2}"/>
     </joint>
     <gazebo reference="pedestal">

Commit message: update moveit_config for new b_bot description

File: homestri_b_bot_moveit_config/config/gazebo_b_bot_scene.urdf (robot description, URDF)
Before this commit: robot b_bot_scene, 27 links, 26 joints
Links:
- removed link closet
- added link camera_bottom_screw_frame
- added link camera_color_frame
- added link camera_color_optical_frame
- added link camera_depth_frame
- added link camera_depth_optical_frame
- added link camera_infra1_frame
- added link camera_infra1_optical_frame
- added link camera_infra2_frame
- added link camera_infra2_optical_frame
- added link camera_link, mass 0.072; collision box size=0.02005 0.099 0.023; visual mesh filename=package://realsense2_description/meshes/d415.stl
- added link realsense_mount, mass 0.0478036670662668; collision mesh filename=package://homestri_description/meshes/components/collision/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 scale=0.001 0.001 0.001; visual mesh filename=package://homestri_description/meshes/components/visual/rea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 scale=0.001 0.001 0.001
- added link wall_1, mass 0.1; collision box size=5 5 0.02
- added link wall_2, mass 0.1; collision box size=5 5 0.02
- added link wall_3, mass 0.1; collision box size=5 5 0.02
Joints:
- removed joint closet_to_world
- added joint camera_color_joint: type fixed, parent camera_link, child camera_color_frame, origin xyz=0 0.015 0 rpy=0 0 0
- added joint camera_color_optical_joint: type fixed, parent camera_color_frame, child camera_color_optical_frame, origin xyz=0 0 0 rpy=-1.5707963267948966 0 -1.5707963267948966
- added joint camera_depth_joint: type fixed, parent camera_link, child camera_depth_frame, origin xyz=0 0 0 rpy=0 0 0
- added joint camera_depth_optical_joint: type fixed, parent camera_depth_frame, child camera_depth_optical_frame, origin xyz=0 0 0 rpy=-1.5707963267948966 0 -1.5707963267948966
- added joint camera_infra1_joint: type fixed, parent camera_link, child camera_infra1_frame, origin xyz=0 0.0 0 rpy=0 0 0
- added joint camera_infra1_optical_joint: type fixed, parent camera_infra1_frame, child camera_infra1_optical_frame, origin xyz=0 0 0 rpy=-1.5707963267948966 0 -1.5707963267948966
- added joint camera_infra2_joint: type fixed, parent camera_link, child camera_infra2_frame, origin xyz=0 -0.055 0 rpy=0 0 0
- added joint camera_infra2_optical_joint: type fixed, parent camera_infra2_frame, child camera_infra2_optical_frame, origin xyz=0 0 0 rpy=-1.5707963267948966 0 -1.5707963267948966
- added joint camera_joint: type fixed, parent realsense_mount, child camera_bottom_screw_frame, origin xyz=0 0.046 0.015 rpy=0 -1.5707963267948966 -1.5707963267948966
- added joint camera_link_joint: type fixed, parent camera_bottom_screw_frame, child camera_link, origin xyz=0 0.02 0.0115 rpy=0 0 0
- added joint realsense_mount_joint: type fixed, parent ee_link, child realsense_mount, origin xyz=0 0 0 rpy=-1.5707963267948966 0 -1.5707963267948966
- added joint wall_1_to_world: type fixed, parent world, child wall_1, origin xyz=0 0 0
- added joint wall_2_to_world: type fixed, parent world, child wall_2, origin xyz=0 0 0
- added joint wall_3_to_world: type fixed, parent world, child wall_3, origin xyz=0 0 0
- joint gripper_tip_link_joint: origin xyz=0.163 0 0 rpy=0 0 0 -> xyz=0.223 0 0 rpy=0 0 0
- joint pedestal_to_world: origin xyz=0 0 0.814 -> xyz=0 0 0.814 rpy=0 0 1.5707963267948966
- joint quick_changer_joint: origin xyz=0 0 0 rpy=1.5707963267948966 0 1.5707963267948966 -> xyz=0 0 0.008 rpy=0 0 3.141592653589793; parent ee_link -> realsense_mount
- joint shoulder_pan_joint: limit lower=-6.283185307179586 upper=6.283185307179586 effort=150.0 velocity=3.141592653589793 -> lower=-3.141592653589793 upper=3.141592653589793 effort=150.0 velocity=3.141592653589793
- joint table_to_world: origin xyz=-1.37 0 0 -> xyz=1.37 0 0
- joint wrist_3_joint: limit lower=-3.141592653589793 upper=3.141592653589793 effort=28.0 velocity=3.141592653589793 -> lower=-6.283185307179586 upper=6.283185307179586 effort=28.0 velocity=3.141592653589793
