Commit message: removed assembly from a_bot scene

File: homestri_description/urdf/workspaces/a_bot_workspace.xacro (robot description, xacro)
@@ -3,5 +3,5 @@
   <xacro:macro name="a_bot_workspace"
     params="pedestal_height:=0.2 pedestal_radius:=0.2 table_height:=0.2 table_y:=0.5 table_x:=0.5">
-    <link name="static_assembly">
+    <!-- <link name="static_assembly">
       <inertial>
         <origin xyz="-0.0019215269775362533 0.02238591812637603 0.00014773610274437554"
@@ -56,5 +56,5 @@
         </geometry>
       </collision>
-    </link>
+    </link> -->
     <link name="pedestal">
       <visual>
@@ -101,5 +101,5 @@
       </inertial>
     </link>
-    <joint name="static_assembly_to_table" type="fixed">
+    <!-- <joint name="static_assembly_to_table" type="fixed">
       <parent link="table" />
       <child link="static_assembly" />
@@ -112,5 +112,5 @@
       <limit effort="1000.0" lower="0" upper=".38" velocity="0.5"/>
       <origin rpy="0 0 0" xyz="0 0 0"/>
-    </joint>
+    </joint> -->
     <joint name="table_to_world" type="fixed">
       <parent link="world" />
