Commit message: fix table physics and placement for b_bot

File: homestri_description/urdf/workspaces/b_bot_workspace.xacro (robot description, xacro)
@@ -29,13 +29,13 @@
     <link name="table">
       <collision>
-        <origin xyz="0 0 .25" rpy="0 0 0" />
+        <origin xyz="0 0 .3" rpy="0 0 0" />
         <geometry>
-          <box size="1 1 0.5" />
+          <box size="1 1 0.6" />
         </geometry>
       </collision>
       <visual>
-        <origin xyz="0 0 .25" rpy="0 0 0" />
+        <origin xyz="0 0 .3" rpy="0 0 0" />
         <geometry>
-          <box size="1 1 0.5" />
+          <box size="1 1 0.6" />
         </geometry>
         <material name="grey">
@@ -44,5 +44,5 @@
       </visual>
       <inertial>
-        <origin xyz="0.0 0.0 0.02" rpy="0 0 0" />
+        <origin xyz="0.0 0.0 0.3" rpy="0 0 0" />
         <mass value=".006784" />
         <inertia ixx=".18e-05" iyy=".18e-05" izz=".18e-05" ixy="0.0" iyz="0.0" ixz="0.0" />
@@ -57,9 +57,4 @@
       </collision>
     </link>
-    <!-- <joint name="pedestal_to_world" type="fixed">
-        <parent link="world"/>
-        <child link="pedestal"/>
-        <origin xyz="0 0 ${pedestal_height}" />
-    </joint> -->
     <joint name="ground_to_world" type="fixed">
       <parent link="world" />
@@ -70,5 +65,5 @@
       <parent link="world" />
       <child link="table" />
-      <origin xyz="1 0 0" />
+      <origin xyz="0 -1 0" />
     </joint>
     <joint name="pedestal_to_world" type="fixed">
@@ -79,4 +74,11 @@
     <gazebo reference="pedestal">
       <material>Gazebo/Grey</material>
+      <selfCollide>true</selfCollide>
+      <kinematic> true </kinematic>
+    </gazebo>
+    <gazebo reference="table">
+      <material>Gazebo/Grey</material>
+      <selfCollide>true</selfCollide>
+      <kinematic> true </kinematic>
     </gazebo>
   </xacro:macro>

Commit message: update b_bot workspace with 4th wall

File: homestri_description/urdf/workspaces/b_bot_workspace.xacro (robot description, xacro)
@@ -82,4 +82,15 @@
       </collision>
     </link>
+    <link name="wall_4">
+      <collision>
+        <origin rpy="${pi/2} 0 0" xyz="0 .98 0" />
+        <geometry>
+          <box size="5 5 0.02" />
+        </geometry>
+        <material name="grey">
+          <color rgba=".5 .5 .5 1.0" />
+        </material>
+      </collision>
+    </link>
     <link name="ground">
       <collision>
@@ -115,4 +126,9 @@
       <origin xyz="0 0 0" />
     </joint>
+    <joint name="wall_4_to_world" type="fixed">
+      <parent link="world" />
+      <child link="wall_4" />
+      <origin xyz="0 0 0" />
+    </joint>
     <joint name="pedestal_to_world" type="fixed">
       <parent link="world" />
