Commit message: simplify workspace, change gripper_tip_link orientation

File: homestri_description/urdf/macros/ur5e_macro.xacro (robot description, xacro)
@@ -41,5 +41,5 @@
       <parent link="${prefix}ee_link" />
       <child link="${prefix}gripper_tip_link" />
-      <origin rpy="0 0 0" xyz="${gripper_tip_offset} 0 0" />
+      <origin rpy="${pi} 0 0" xyz="${gripper_tip_offset} 0 0" />
     </joint>
     <!-- ############ GAZEBO PROPERTIES ############ -->

File: homestri_description/urdf/workspaces/a_bot_workspace.xacro (robot description, xacro)
@@ -79,5 +79,5 @@
       </inertial>
     </link>
-    <link name="table">
+    <!-- <link name="table">
       <collision>
         <origin xyz="0 -0.31 ${-table_height/2}" rpy="0 0 0" />
@@ -100,5 +100,5 @@
         <inertia ixx=".18e-05" iyy=".18e-05" izz=".18e-05" ixy="0.0" iyz="0.0" ixz="0.0" />
       </inertial>
-    </link>
+    </link> -->
     <!-- <joint name="static_assembly_to_table" type="fixed">
       <parent link="table" />
@@ -113,9 +113,9 @@
       <origin rpy="0 0 0" xyz="0 0 0"/>
     </joint> -->
-    <joint name="table_to_world" type="fixed">
+    <!-- <joint name="table_to_world" type="fixed">
       <parent link="world" />
       <child link="table" />
       <origin xyz="${table_x} ${table_y} ${table_height}" />
-    </joint>
+    </joint> -->
     <joint name="pedestal_to_world" type="fixed">
       <parent link="world" />
