Commit message: fix docker, remove unnecessary pkgs, refactor homestri_description

File: catkin_ws/src/homestri-ur/homestri_description/urdf/macros/ur5e_macro.xacro (robot description, xacro)
@@ -3,10 +3,16 @@
 <!-- The position of the TF frame has not been measured at all and needs to be calibrated. -->
 <robot name="ur5e" xmlns:xacro="http://www.ros.org/wiki/xacro">
-  <xacro:macro name="ur5e" params="prefix parent transmission_hw_interface gripper_tip_offset *origin">
+  <xacro:macro name="ur5e" params="
+    prefix
+    parent
+    transmission_hw_interface:=hardware_interface/PositionJointInterface
+    joint_limits_parameters_file:='$(find ur_description)/config/ur5e/joint_limits.yaml'
+    tcp_offset
+    *origin">
     <!-- ur5e -->
     <xacro:include filename="$(find ur_description)/urdf/inc/ur_macro.xacro" />
     <xacro:ur_robot
       prefix="${prefix}"
-      joint_limits_parameters_file='$(find homestri_description)/config/ur5e_joint_limits.yaml'
+      joint_limits_parameters_file="${joint_limits_parameters_file}"
       kinematics_parameters_file='$(find ur_description)/config/ur5e/default_kinematics.yaml'
       physical_parameters_file='$(find ur_description)/config/ur5e/physical_parameters.yaml'
@@ -22,69 +28,11 @@
       <xacro:insert_block name="origin" />
     </joint>
-    <!-- end effector link -->
-    <link name="${prefix}ee_link">
-      <collision>
-        <geometry>
-          <box size="0.01 0.01 0.01" />
-        </geometry>
-        <origin rpy="0 0 0" xyz="-0.01 0 0" />
-      </collision>
-    </link>
-    <joint name="${prefix}ee_fixed_joint" type="fixed">
+    <!-- Add an additional link to plan with. Oriented like the UR ee_link frame. -->
+    <link name="${prefix}tcp_link" />
+    <joint name="${prefix}tcp_joint" type="fixed">
       <parent link="${prefix}wrist_3_link" />
-      <child link="${prefix}ee_link" />
-      <origin rpy="0.0 -1.57079632679 1.57079632679" xyz="0.0 0.0 0.0" />
+      <child link="${prefix}tcp_link" />
+      <origin rpy="0 ${-pi/2} ${-pi/2}" xyz="0 0 ${tcp_offset}" />
     </joint>
-    <!-- Add an additional link to plan with. Oriented like the UR ee_link frame. -->
-    <link name="${prefix}gripper_tip_link" />
-    <joint name="${prefix}gripper_tip_link_joint" type="fixed">
-      <parent link="${prefix}ee_link" />
-      <child link="${prefix}gripper_tip_link" />
-      <origin rpy="0 0 0" xyz="${gripper_tip_offset} 0 0" />
-    </joint>
-    <!-- ############ GAZEBO PROPERTIES ############ -->
-    <gazebo reference="${prefix}wrist_3_joint">
-        <provideFeedback>true</provideFeedback>
-    </gazebo>
-    <gazebo>
-      <plugin filename="libgazebo_ros_ft_sensor.so" name="ft_sensor">
-        <updateRate>100.0</updateRate>
-        <topicName>wrench</topicName>
-        <jointName>${prefix}wrist_3_joint</jointName>
-        <!-- <noise>
-          <type>gaussian</type>
-          <mean>0.0</mean>
-          <stddev>0.003</stddev>
-        </noise> -->
-      </plugin>
-    </gazebo>
-    <xacro:macro name="ur5e_gazebo_link_properties" params="reference">
-      <gazebo reference="${reference}">
-        <kp>1000000.0</kp>
-        <kd>1.0</kd>
-        <mu1>0.8</mu1>
-        <mu2>0.8</mu2>
-        <maxVel>0.0</maxVel>
-        <minDepth>0.001</minDepth>
-        <selfCollide>true</selfCollide>
-      </gazebo>
-    </xacro:macro>
-    <xacro:ur5e_gazebo_link_properties reference="${prefix}shoulder_link" />
-    <xacro:ur5e_gazebo_link_properties reference="${prefix}upper_arm_link" />
-    <xacro:ur5e_gazebo_link_properties reference="${prefix}forearm_link" />
-    <xacro:ur5e_gazebo_link_properties reference="${prefix}wrist_1_link" />
-    <xacro:ur5e_gazebo_link_properties reference="${prefix}wrist_2_link" />
-    <xacro:ur5e_gazebo_link_properties reference="${prefix}wrist_3_link" />
-    <xacro:macro name="ur5e_gazebo_joint_properties" params="reference">
-      <gazebo reference="${reference}">
-        <implicitSpringDamper>true</implicitSpringDamper>
-      </gazebo>
-    </xacro:macro>
-    <xacro:ur5e_gazebo_link_properties reference="${prefix}shoulder_pan_joint" />
-    <xacro:ur5e_gazebo_link_properties reference="${prefix}shoulder_lift_joint" />
-    <xacro:ur5e_gazebo_link_properties reference="${prefix}elbow_joint" />
-    <xacro:ur5e_gazebo_link_properties reference="${prefix}wrist_1_joint" />
-    <xacro:ur5e_gazebo_link_properties reference="${prefix}wrist_2_joint" />
-    <xacro:ur5e_gazebo_link_properties reference="${prefix}wrist_3_joint" />
   </xacro:macro>
 </robot>

File: catkin_ws/src/homestri-ur/homestri_description/urdf/scenes/a_bot_scene.xacro (robot description, xacro)
@@ -1,30 +1,21 @@
 <?xml version="1.0"?>
 <robot xmlns:xacro="http://www.ros.org/wiki/xacro" name="a_bot_scene">
-    <xacro:include filename="$(find homestri_description)/urdf/workspaces/a_bot_workspace.xacro" />
-    <xacro:include filename="$(find homestri_description)/urdf/macros/ur5e_macro.xacro" />
-    <xacro:include
-        filename="$(find homestri_description)/urdf/macros/robotiq_realsense_macro.xacro" />
-    <xacro:a_bot_workspace
+    <xacro:arg name="joint_limits_parameters_file"
+        default="$(find ur_description)/config/ur5e/joint_limits.yaml" />
+    <xacro:arg name="transmission_hw_interface" default="hardware_interface/PositionJointInterface" />
+    <xacro:include filename="$(find homestri_description)/urdf/workspaces/pedestal_workspace.xacro" />
+    <xacro:include filename="$(find homestri_description)/urdf/macros/a_bot_macro.xacro" />
+    <xacro:pedestal_workspace
         pedestal_height="0.6"
         pedestal_radius="0.15"
-        table_height="0.4"
-        table_y="-0.8"
-        table_x="0.25"
     />
-    <xacro:ur5e
+    <xacro:a_bot
         prefix=""
         parent="pedestal"
-        gripper_tip_offset="0.163"
-        transmission_hw_interface="hardware_interface/PositionJointInterface"
+        transmission_hw_interface="$(arg transmission_hw_interface)"
+        joint_limits_parameters_file="$(arg joint_limits_parameters_file)"
     >
         <origin xyz="0 0 0" rpy="0 0 0" />
-    </xacro:ur5e>
-    <xacro:robotiq_realsense
-        prefix=""
-        parent="ee_link"
-        transmission_hw_interface="hardware_interface/PositionJointInterface"
-    >
-        <origin xyz="0 0 0" rpy="${-pi/2} ${0} ${-pi/2}" />
-    </xacro:robotiq_realsense>
+    </xacro:a_bot>
     <link name="world" />
     <gazebo>

File: catkin_ws/src/homestri-ur/homestri_description/urdf/scenes/b_bot_scene.xacro (robot description, xacro)
@@ -1,24 +1,21 @@
 <?xml version="1.0"?>
 <robot xmlns:xacro="http://www.ros.org/wiki/xacro" name="b_bot_scene">
-    <xacro:include filename="$(find homestri_description)/urdf/workspaces/b_bot_workspace.xacro" />
-    <xacro:include filename="$(find homestri_description)/urdf/macros/ur5e_macro.xacro" />
-    <xacro:include
-        filename="$(find homestri_description)/urdf/macros/onrobot_realsense_macro.xacro" />
-    <xacro:b_bot_workspace />
-    <xacro:ur5e
+    <xacro:arg name="joint_limits_parameters_file"
+        default="$(find ur_description)/config/ur5e/joint_limits.yaml" />
+    <xacro:arg name="transmission_hw_interface" default="hardware_interface/PositionJointInterface" />
+    <xacro:include filename="$(find homestri_description)/urdf/workspaces/pedestal_workspace.xacro" />
+    <xacro:include filename="$(find homestri_description)/urdf/macros/b_bot_macro.xacro" />
+    <xacro:pedestal_workspace
+        pedestal_height="0.6"
+        pedestal_radius="0.15"
+    />
+    <xacro:b_bot
         prefix=""
         parent="pedestal"
-        gripper_tip_offset="0.223"
-        transmission_hw_interface="hardware_interface/PositionJointInterface"
+        transmission_hw_interface="$(arg transmission_hw_interface)"
+        joint_limits_parameters_file="$(arg joint_limits_parameters_file)"
     >
         <origin xyz="0 0 0" rpy="0 0 0" />
-    </xacro:ur5e>
-    <xacro:onrobot_realsense
-        prefix=""
-        parent="ee_link"
-        transmission_hw_interface="hardware_interface/PositionJointInterface"
-    >
-        <origin xyz="0 0 0" rpy="${-pi/2} ${0} ${-pi/2}" />
-    </xacro:onrobot_realsense>
+    </xacro:b_bot>
     <link name="world" />
     <gazebo>
