Commit message: clean up moveit configs and gazebo

File: catkin_ws/src/homestri-ur/homestri_a_bot_moveit_config/config/gazebo_a_bot_scene.urdf (robot description, URDF)
Before this commit: robot a_bot_scene, 42 links, 41 joints
Links:
- removed link ee_link
- removed link gripper_tip_link
- removed link moving_assembly
- removed link realsense_mount
- removed link static_assembly
- removed link table
- added link d415_mount_attach_link
- added link d415_mount_link, mass 0.0478036670662668; collision mesh filename=package://homestri_description/meshes/collision/d415_mount.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 scale=0.001 0.001 0.001; visual mesh filename=package://homestri_description/meshes/visual/d415_mount.stl scale=0.001 0.001 0.001
- added link tcp_link
- link pedestal: geometry collision cylinder length=0.6 radius=0.15; visual cylinder length=0.6 radius=0.15
Joints:
- removed joint ee_fixed_joint
- removed joint gripper_tip_link_joint
- removed joint moving_assembly_joint
- removed joint pedestal_to_world
- removed joint realsense_mount_joint
- removed joint static_assembly_to_table
- removed joint table_to_world
- added joint d415_mount_attach_joint: type fixed, parent d415_mount_link, child d415_mount_attach_link, origin xyz=0 0 0.005 rpy=0 0 0
- added joint d415_mount_joint: type fixed, parent wrist_3_link, child d415_mount_link, origin xyz=0 0 0 rpy=0 0 0
- added joint pedestal_joint: type fixed, parent world, child pedestal, origin xyz=0 0 0.6
- added joint tcp_joint: type fixed, parent wrist_3_link, child tcp_link, origin xyz=0 0 0.163 rpy=0 -1.5707963267948966 -1.5707963267948966
- joint camera_joint: parent realsense_mount -> d415_mount_link
- joint coupler_joint: origin xyz=0 0 0.008 rpy=0 0 3.141592653589793 -> xyz=0 0 0.003 rpy=0 0 3.141592653589793; parent realsense_mount -> d415_mount_attach_link
- joint elbow_joint: limit lower=0.0 upper=3.141592653589793 effort=150.0 velocity=3.141592653589793 -> lower=-3.141592653589793 upper=3.141592653589793 effort=150.0 velocity=3.141592653589793
- joint shoulder_lift_joint: limit lower=-3.141592653589793 upper=3.141592653589793 effort=150.0 velocity=3.141592653589793 -> lower=-6.283185307179586 upper=6.283185307179586 effort=150.0 velocity=3.141592653589793
- joint shoulder_pan_joint: limit lower=-3.141592653589793 upper=3.141592653589793 effort=150.0 velocity=3.141592653589793 -> lower=-6.283185307179586 upper=6.283185307179586 effort=150.0 velocity=3.141592653589793
- joint wrist_1_joint: limit lower=-3.141592653589793 upper=3.141592653589793 effort=28.0 velocity=3.141592653589793 -> lower=-6.283185307179586 upper=6.283185307179586 effort=28.0 velocity=3.141592653589793
- joint wrist_2_joint: limit lower=-3.141592653589793 upper=3.141592653589793 effort=28.0 velocity=3.141592653589793 -> lower=-6.283185307179586 upper=6.283185307179586 effort=28.0 velocity=3.141592653589793
- joint wrist_3_joint: limit lower=0.0 upper=6.283185307179586 effort=28.0 velocity=3.141592653589793 -> lower=-6.283185307179586 upper=6.283185307179586 effort=28.0 velocity=3.141592653589793

File: catkin_ws/src/homestri-ur/homestri_b_bot_moveit_config/config/gazebo_b_bot_scene.urdf (robot description, URDF)
Before this commit: robot b_bot_scene, 40 links, 39 joints
Links:
- removed link ee_link
- removed link gripper_tip_link
- removed link ground
- removed link realsense_mount
- removed link table
- removed link wall_1
- removed link wall_2
- removed link wall_3
- added link d415_mount_attach_link
- added link d415_mount_link, mass 0.0478036670662668; collision mesh filename=package://homestri_description/meshes/collision/d415_mount.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 scale=0.001 0.001 0.001; visual mesh filename=package://homestri_description/meshes/visual/d415_mount.stl scale=0.001 0.001 0.001
- added link tcp_link
- link pedestal: geometry collision cylinder length=0.6 radius=0.15; visual cylinder length=0.6 radius=0.15
Joints:
- removed joint ee_fixed_joint
- removed joint gripper_tip_link_joint
- removed joint ground_to_world
- removed joint pedestal_to_world
- removed joint realsense_mount_joint
- removed joint table_to_world
- removed joint wall_1_to_world
- removed joint wall_2_to_world
- removed joint wall_3_to_world
- added joint d415_mount_attach_joint: type fixed, parent d415_mount_link, child d415_mount_attach_link, origin xyz=0 0 0.005 rpy=0 0 0
- added joint d415_mount_joint: type fixed, parent wrist_3_link, child d415_mount_link, origin xyz=0 0 0 rpy=0 0 0
- added joint pedestal_joint: type fixed, parent world, child pedestal, origin xyz=0 0 0.6
- added joint tcp_joint: type fixed, parent wrist_3_link, child tcp_link, origin xyz=0 0 0.223 rpy=0 -1.5707963267948966 -1.5707963267948966
- joint camera_joint: parent realsense_mount -> d415_mount_link
- joint elbow_joint: limit lower=0.0 upper=3.141592653589793 effort=150.0 velocity=3.141592653589793 -> lower=-3.141592653589793 upper=3.141592653589793 effort=150.0 velocity=3.141592653589793
- joint quick_changer_joint: origin xyz=0 0 0.008 rpy=0 0 3.141592653589793 -> xyz=0 0 0.0026 rpy=0 0 3.141592653589793; parent realsense_mount -> d415_mount_attach_link
- joint shoulder_lift_joint: limit lower=-3.141592653589793 upper=3.141592653589793 effort=150.0 velocity=3.141592653589793 -> lower=-6.283185307179586 upper=6.283185307179586 effort=150.0 velocity=3.141592653589793
- joint shoulder_pan_joint: limit lower=-3.141592653589793 upper=3.141592653589793 effort=150.0 velocity=3.141592653589793 -> lower=-6.283185307179586 upper=6.283185307179586 effort=150.0 velocity=3.141592653589793
- joint wrist_1_joint: limit lower=-3.141592653589793 upper=3.141592653589793 effort=28.0 velocity=3.141592653589793 -> lower=-6.283185307179586 upper=6.283185307179586 effort=28.0 velocity=3.141592653589793
- joint wrist_2_joint: limit lower=-3.141592653589793 upper=3.141592653589793 effort=28.0 velocity=3.141592653589793 -> lower=-6.283185307179586 upper=6.283185307179586 effort=28.0 velocity=3.141592653589793
